File: pcb/decoupling.sch (KiCad schematic (older format))
At the start: 6 parts

Commit message: lagt til SPI
Parts:
- gave numbers to parts that had none: 6
Changed lines of the file:
@@
 $EndDescr
 $Comp
-L Device:C C?
+L Device:C C1
 U 1 1 5BA59925
 P 4700 3850
-F 0 "C?" H 4815 3896 50  0000 L CNN
+F 0 "C1" H 4815 3896 50  0000 L CNN
 F 1 "100n" H 4815 3805 50  0000 L CNN
 F 2 "" H 4738 3700 50  0001 C CNN
@@
 $EndComp
 $Comp
-L Device:C C?
+L Device:C C2
 U 1 1 5BA59950
 P 5050 3850
-F 0 "C?" H 5165 3896 50  0000 L CNN
+F 0 "C2" H 5165 3896 50  0000 L CNN
 F 1 "100n" H 5165 3805 50  0000 L CNN
 F 2 "" H 5088 3700 50  0001 C CNN
@@
 $EndComp
 $Comp
-L Device:C C?
+L Device:C C3
 U 1 1 5BA5996E
 P 5400 3850
-F 0 "C?" H 5515 3896 50  0000 L CNN
+F 0 "C3" H 5515 3896 50  0000 L CNN
 F 1 "100n" H 5515 3805 50  0000 L CNN
 F 2 "" H 5438 3700 50  0001 C CNN
@@
 $EndComp
 $Comp
-L Device:C C?
+L Device:C C4
 U 1 1 5BA599BB
 P 5750 3850
-F 0 "C?" H 5865 3896 50  0000 L CNN
+F 0 "C4" H 5865 3896 50  0000 L CNN
 F 1 "100n" H 5865 3805 50  0000 L CNN
 F 2 "" H 5788 3700 50  0001 C CNN
@@
 $EndComp
 $Comp
-L Device:C C?
+L Device:C C5
 U 1 1 5BA599F7
 P 6100 3850
-F 0 "C?" H 6215 3896 50  0000 L CNN
+F 0 "C5" H 6215 3896 50  0000 L CNN
 F 1 "100n" H 6215 3805 50  0000 L CNN
 F 2 "" H 6138 3700 50  0001 C CNN
@@
 $EndComp
 $Comp
-L Device:C C?
+L Device:C C6
 U 1 1 5BA59A1B
 P 6450 3850
-F 0 "C?" H 6565 3896 50  0000 L CNN
+F 0 "C6" H 6565 3896 50  0000 L CNN
 F 1 "10u" H 6565 3805 50  0000 L CNN
 F 2 "" H 6488 3700 50  0001 C CNN
@@
 	1    0    0    -1
 $EndComp
-Text GLabel 4100 3700 0    50   Input ~ 0
-VDD_DEC
-Text GLabel 4100 4000 0    50   Input ~ 0
-VSS_DEC
 $Comp
-L power:+3.3V #PWR?
+L power:+3.3V #PWR0127
 U 1 1 5BA5C380
 P 6450 3550
-F 0 "#PWR?" H 6450 3400 50  0001 C CNN
+F 0 "#PWR0127" H 6450 3400 50  0001 C CNN
 F 1 "+3.3V" H 6465 3723 50  0000 C CNN
 F 2 "" H 6450 3550 50  0001 C CNN
@@
 $EndComp
 $Comp
-L power:GND #PWR?
+L power:GND #PWR0128
 U 1 1 5BA5C3F3
 P 6450 4150
-F 0 "#PWR?" H 6450 3900 50  0001 C CNN
+F 0 "#PWR0128" H 6450 3900 50  0001 C CNN
 F 1 "GND" H 6455 3977 50  0000 C CNN
 F 2 "" H 6450 4150 50  0001 C CNN
@@
 Wire Wire Line
 	6100 4000 5750 4000
+Text HLabel 4100 3700 0    50   Input ~ 0
+VDD_DEC
+Text HLabel 4100 4000 0    50   Input ~ 0
+VSS_DEC
 $EndSCHEMATC

Commit message: Prettyfy Schematic
Parts:
- added C10, C7: 1uF, symbol Device:C
- added C2, C5: 10nF, symbol Device:C
- added L1: 742792662, symbol Device:L
- added R5: 1, symbol Device:R
- renumbered C2 to C3, C3 to C4, C4 to C6, C5 to C8, C6 to C9
Connections:
- net labels added: AVDD_DEC, DEC
- wire segments 14 -> 25
