File: pcb/OLD-SONAR.sch (KiCad schematic (older format))
At the start: 14 parts

Commit message: Finishe schematic, add netlist and start editing pcb design
Parts:
- Q1, Q2, Q3, Q4: renamed from Q?; footprint Package_TO_SOT_SMD:SOT-23 -> digikey-footprints:SOT-23-3
- R10, R11, R12, R13, R6, R7, R8, R9: renamed from R?; footprint (none) -> Resistor_SMD:R_0603_1608Metric_Pad1.05x0.95mm_HandSolder
- U5, U6: renamed from U?; footprint (none) -> Connector_PinHeader_2.54mm:PinHeader_1x04_P2.54mm_Vertical
Changed lines of the file:
@@
 $Descr A4 11693 8268
 encoding utf-8
-Sheet 10 10
+Sheet 9 10
 Title ""
 Date ""
@@
 P 3300 5200
 AR Path="/5BAA6CA9/5BAB9F55" Ref="R?"  Part="1"
-AR Path="/5BAB97A9/5BAB9F55" Ref="R?"  Part="1"
-F 0 "R?" H 3370 5246 50  0000 L CNN
+AR Path="/5BAB97A9/5BAB9F55" Ref="R7"  Part="1"
+F 0 "R7" H 3370 5246 50  0000 L CNN
 F 1 "10k" H 3370 5155 50  0000 L CNN
-F 2 "" V 3230 5200 50  0001 C CNN
+F 2 "Resistor_SMD:R_0603_1608Metric_Pad1.05x0.95mm_HandSolder" V 3230 5200 50  0001 C CNN
 F 3 "~" H 3300 5200 50  0001 C CNN
 	1    3300 5200
@@
 P 3300 4550
 AR Path="/5BAA6CA9/5BAB9F5C" Ref="R?"  Part="1"
-AR Path="/5BAB97A9/5BAB9F5C" Ref="R?"  Part="1"
-F 0 "R?" H 3370 4596 50  0000 L CNN
+AR Path="/5BAB97A9/5BAB9F5C" Ref="R6"  Part="1"
+F 0 "R6" H 3370 4596 50  0000 L CNN
 F 1 "10k" H 3370 4505 50  0000 L CNN
-F 2 "" V 3230 4550 50  0001 C CNN
+F 2 "Resistor_SMD:R_0603_1608Metric_Pad1.05x0.95mm_HandSolder" V 3230 4550 50  0001 C CNN
 F 3 "~" H 3300 4550 50  0001 C CNN
 	1    3300 4550
@@
 P 3550 4850
 AR Path="/5BAA6CA9/5BAB9F8D" Ref="Q?"  Part="1"
-AR Path="/5BAB97A9/5BAB9F8D" Ref="Q?"  Part="1"
-F 0 "Q?" V 3800 4850 50  0000 C CNN
+AR Path="/5BAB97A9/5BAB9F8D" Ref="Q1"  Part="1"
+F 0 "Q1" V 3800 4850 50  0000 C CNN
 F 1 "BSS138" V 3891 4850 50  0000 C CNN
-F 2 "Package_TO_SOT_SMD:SOT-23" H 3750 4775 50  0001 L CIN
+F 2 "digikey-footprints:SOT-23-3" H 3750 4775 50  0001 L CIN
 F 3 "https://www.fairchildsemi.com/datasheets/BS/BSS138.pdf" H 3550 4850 50  0001 L CNN
 	1    3550 4850
@@
 	3350 4950 3350 4850
 $Comp
-L localization-symbols:HC-SR04 U?
+L localization-symbols:HC-SR04 U5
 U 1 1 5BABA401
 P 4500 3500
-F 0 "U?" H 4728 3515 50  0000 L CNN
+F 0 "U5" H 4728 3515 50  0000 L CNN
 F 1 "HC-SR04" H 4728 3424 50  0000 L CNN
-F 2 "" H 4500 3350 50  0001 C CNN
+F 2 "Connector_PinHeader_2.54mm:PinHeader_1x04_P2.54mm_Vertical" H 4500 3350 50  0001 C CNN
 F 3 "" H 4500 3350 50  0001 C CNN
 	1    4500 3500
@@
 $EndComp
 $Comp
-L power:+3.3V #PWR?
+L power:+3.3V #PWR02
 U 1 1 5BABB70B
 P 2950 5200
-F 0 "#PWR?" H 2950 5050 50  0001 C CNN
+F 0 "#PWR02" H 2950 5050 50  0001 C CNN
 F 1 "+3.3V" H 2965 5373 50  0000 C CNN
 F 2 "" H 2950 5200 50  0001 C CNN
@@
 $EndComp
 $Comp
-L power:VCC #PWR?
+L power:VCC #PWR01
 U 1 1 5BABC095
 P 2950 4550
-F 0 "#PWR?" H 2950 4400 50  0001 C CNN
+F 0 "#PWR01" H 2950 4400 50  0001 C CNN
 F 1 "VCC" H 2968 4723 50  0000 C CNN
 F 2 "" H 2950 4550 50  0001 C CNN
@@
 $EndComp
 $Comp
-L power:VCC #PWR?
+L power:VCC #PWR029
 U 1 1 5BABC2C1
 P 4350 3700
-F 0 "#PWR?" H 4350 3550 50  0001 C CNN
+F 0 "#PWR029" H 4350 3550 50  0001 C CNN
 F 1 "VCC" H 4368 3873 50  0000 C CNN
 F 2 "" H 4350 3700 50  0001 C CNN
@@
 $EndComp
 $Comp
-L power:GND #PWR?
+L power:GND #PWR032
 U 1 1 5BABC33B
 P 4650 3700
-F 0 "#PWR?" H 4650 3450 50  0001 C CNN
+F 0 "#PWR032" H 4650 3450 50  0001 C CNN
 F 1 "GND" H 4655 3527 50  0000 C CNN
 F 2 "" H 4650 3700 50  0001 C CNN
@@
 P 4700 5200
 AR Path="/5BAA6CA9/5BABCF71" Ref="R?"  Part="1"
-AR Path="/5BAB97A9/5BABCF71" Ref="R?"  Part="1"
-F 0 "R?" H 4770 5246 50  0000 L CNN
+AR Path="/5BAB97A9/5BABCF71" Ref="R9"  Part="1"
+F 0 "R9" H 4770 5246 50  0000 L CNN
 F 1 "10k" H 4770 5155 50  0000 L CNN
-F 2 "" V 4630 5200 50  0001 C CNN
+F 2 "Resistor_SMD:R_0603_1608Metric_Pad1.05x0.95mm_HandSolder" V 4630 5200 50  0001 C CNN
 F 3 "~" H 4700 5200 50  0001 C CNN
 	1    4700 5200
@@
 P 4700 4550
 AR Path="/5BAA6CA9/5BABCF78" Ref="R?"  Part="1"
-AR Path="/5BAB97A9/5BABCF78" Ref="R?"  Part="1"
-F 0 "R?" H 4770 4596 50  0000 L CNN
+AR Path="/5BAB97A9/5BABCF78" Ref="R8"  Part="1"
+F 0 "R8" H 4770 4596 50  0000 L CNN
 F 1 "10k" H 4770 4505 50  0000 L CNN
-F 2 "" V 4630 4550 50  0001 C CNN
+F 2 "Resistor_SMD:R_0603_1608Metric_Pad1.05x0.95mm_HandSolder" V 4630 4550 50  0001 C CNN
 F 3 "~" H 4700 4550 50  0001 C CNN
 	1    4700 4550
@@
 P 4950 4850
 AR Path="/5BAA6CA9/5BABCF8C" Ref="Q?"  Part="1"
-AR Path="/5BAB97A9/5BABCF8C" Ref="Q?"  Part="1"
-F 0 "Q?" V 5200 4850 50  0000 C CNN
+AR Path="/5BAB97A9/5BABCF8C" Ref="Q2"  Part="1"
+F 0 "Q2" V 5200 4850 50  0000 C CNN
 F 1 "BSS138" V 5291 4850 50  0000 C CNN
-F 2 "Package_TO_SOT_SMD:SOT-23" H 5150 4775 50  0001 L CIN
+F 2 "digikey-footprints:SOT-23-3" H 5150 4775 50  0001 L CIN
 F 3 "https://www.fairchildsemi.com/datasheets/BS/BSS138.pdf" H 4950 4850 50  0001 L CNN
 	1    4950 4850
@@
 	4750 4950 4750 4850
 $Comp
-L power:+3.3V #PWR?
+L power:+3.3V #PWR031
 U 1 1 5BABCF94
 P 4350 5200
-F 0 "#PWR?" H 4350 5050 50  0001 C CNN
+F 0 "#PWR031" H 4350 5050 50  0001 C CNN
 F 1 "+3.3V" H 4365 5373 50  0000 C CNN
 F 2 "" H 4350 5200 50  0001 C CNN
@@
 $EndComp
 $Comp
-L power:VCC #PWR?
+L power:VCC #PWR030
 U 1 1 5BABCF9A
 P 4350 4550
-F 0 "#PWR?" H 4350 4400 50  0001 C CNN
+F 0 "#PWR030" H 4350 4400 50  0001 C CNN
 F 1 "VCC" H 4368 4723 50  0000 C CNN
 F 2 "" H 4350 4550 50  0001 C CNN
@@
 P 6200 5200
 AR Path="/5BAA6CA9/5BABDC8E" Ref="R?"  Part="1"
-AR Path="/5BAB97A9/5BABDC8E" Ref="R?"  Part="1"
-F 0 "R?" H 6270 5246 50  0000 L CNN
+AR Path="/5BAB97A9/5BABDC8E" Ref="R11"  Part="1"
+F 0 "R11" H 6270 5246 50  0000 L CNN
 F 1 "10k" H 6270 5155 50  0000 L CNN
-F 2 "" V 6130 5200 50  0001 C CNN
+F 2 "Resistor_SMD:R_0603_1608Metric_Pad1.05x0.95mm_HandSolder" V 6130 5200 50  0001 C CNN
 F 3 "~" H 6200 5200 50  0001 C CNN
 	1    6200 5200
@@
 P 6200 4550
 AR Path="/5BAA6CA9/5BABDC95" Ref="R?"  Part="1"
-AR Path="/5BAB97A9/5BABDC95" Ref="R?"  Part="1"
-F 0 "R?" H 6270 4596 50  0000 L CNN
+AR Path="/5BAB97A9/5BABDC95" Ref="R10"  Part="1"
+F 0 "R10" H 6270 4596 50  0000 L CNN
 F 1 "10k" H 6270 4505 50  0000 L CNN
-F 2 "" V 6130 4550 50  0001 C CNN
+F 2 "Resistor_SMD:R_0603_1608Metric_Pad1.05x0.95mm_HandSolder" V 6130 4550 50  0001 C CNN
 F 3 "~" H 6200 4550 50  0001 C CNN
 	1    6200 4550
@@
 P 6450 4850
 AR Path="/5BAA6CA9/5BABDCA8" Ref="Q?"  Part="1"
-AR Path="/5BAB97A9/5BABDCA8" Ref="Q?"  Part="1"
-F 0 "Q?" V 6700 4850 50  0000 C CNN
+AR Path="/5BAB97A9/5BABDCA8" Ref="Q3"  Part="1"
+F 0 "Q3" V 6700 4850 50  0000 C CNN
 F 1 "BSS138" V 6791 4850 50  0000 C CNN
-F 2 "Package_TO_SOT_SMD:SOT-23" H 6650 4775 50  0001 L CIN
+F 2 "digikey-footprints:SOT-23-3" H 6650 4775 50  0001 L CIN
 F 3 "https://www.fairchildsemi.com/datasheets/BS/BSS138.pdf" H 6450 4850 50  0001 L CNN
 	1    6450 4850
@@
 	6250 4950 6250 4850
 $Comp
-L localization-symbols:HC-SR04 U?
+L localization-symbols:HC-SR04 U6
 U 1 1 5BABDCB0
 P 7400 3500
-F 0 "U?" H 7628 3515 50  0000 L CNN
+F 0 "U6" H 7628 3515 50  0000 L CNN
 F 1 "HC-SR04" H 7628 3424 50  0000 L CNN
-F 2 "" H 7400 3350 50  0001 C CNN
+F 2 "Connector_PinHeader_2.54mm:PinHeader_1x04_P2.54mm_Vertical" H 7400 3350 50  0001 C CNN
 F 3 "" H 7400 3350 50  0001 C CNN
 	1    7400 3500
@@
 $EndComp
 $Comp
-L power:+3.3V #PWR?
+L power:+3.3V #PWR034
 U 1 1 5BABDCB7
 P 5850 5200
-F 0 "#PWR?" H 5850 5050 50  0001 C CNN
+F 0 "#PWR034" H 5850 5050 50  0001 C CNN
 F 1 "+3.3V" H 5865 5373 50  0000 C CNN
 F 2 "" H 5850 5200 50  0001 C CNN
@@
 $EndComp
 $Comp
-L power:VCC #PWR?
+L power:VCC #PWR033
 U 1 1 5BABDCBD
 P 5850 4550
-F 0 "#PWR?" H 5850 4400 50  0001 C CNN
+F 0 "#PWR033" H 5850 4400 50  0001 C CNN
 F 1 "VCC" H 5868 4723 50  0000 C CNN
 F 2 "" H 5850 4550 50  0001 C CNN
@@
 $EndComp
 $Comp
-L power:VCC #PWR?
+L power:VCC #PWR035
 U 1 1 5BABDCC3
 P 7250 3700
-F 0 "#PWR?" H 7250 3550 50  0001 C CNN
+F 0 "#PWR035" H 7250 3550 50  0001 C CNN
 F 1 "VCC" H 7268 3873 50  0000 C CNN
 F 2 "" H 7250 3700 50  0001 C CNN
@@
 $EndComp
 $Comp
-L power:GND #PWR?
+L power:GND #PWR038
 U 1 1 5BABDCC9
 P 7550 3700
-F 0 "#PWR?" H 7550 3450 50  0001 C CNN
+F 0 "#PWR038" H 7550 3450 50  0001 C CNN
 F 1 "GND" H 7555 3527 50  0000 C CNN
 F 2 "" H 7550 3700 50  0001 C CNN
@@
 P 7600 5200
 AR Path="/5BAA6CA9/5BABDCCF" Ref="R?"  Part="1"
-AR Path="/5BAB97A9/5BABDCCF" Ref="R?"  Part="1"
-F 0 "R?" H 7670 5246 50  0000 L CNN
+AR Path="/5BAB97A9/5BABDCCF" Ref="R13"  Part="1"
+F 0 "R13" H 7670 5246 50  0000 L CNN
 F 1 "10k" H 7670 5155 50  0000 L CNN
-F 2 "" V 7530 5200 50  0001 C CNN
+F 2 "Resistor_SMD:R_0603_1608Metric_Pad1.05x0.95mm_HandSolder" V 7530 5200 50  0001 C CNN
 F 3 "~" H 7600 5200 50  0001 C CNN
 	1    7600 5200
@@
 P 7600 4550
 AR Path="/5BAA6CA9/5BABDCD6" Ref="R?"  Part="1"
-AR Path="/5BAB97A9/5BABDCD6" Ref="R?"  Part="1"
-F 0 "R?" H 7670 4596 50  0000 L CNN
+AR Path="/5BAB97A9/5BABDCD6" Ref="R12"  Part="1"
+F 0 "R12" H 7670 4596 50  0000 L CNN
 F 1 "10k" H 7670 4505 50  0000 L CNN
-F 2 "" V 7530 4550 50  0001 C CNN
+F 2 "Resistor_SMD:R_0603_1608Metric_Pad1.05x0.95mm_HandSolder" V 7530 4550 50  0001 C CNN
 F 3 "~" H 7600 4550 50  0001 C CNN
 	1    7600 4550
@@
 P 7850 4850
 AR Path="/5BAA6CA9/5BABDCE9" Ref="Q?"  Part="1"
-AR Path="/5BAB97A9/5BABDCE9" Ref="Q?"  Part="1"
-F 0 "Q?" V 8100 4850 50  0000 C CNN
+AR Path="/5BAB97A9/5BABDCE9" Ref="Q4"  Part="1"
+F 0 "Q4" V 8100 4850 50  0000 C CNN
 F 1 "BSS138" V 8191 4850 50  0000 C CNN
-F 2 "Package_TO_SOT_SMD:SOT-23" H 8050 4775 50  0001 L CIN
+F 2 "digikey-footprints:SOT-23-3" H 8050 4775 50  0001 L CIN
 F 3 "https://www.fairchildsemi.com/datasheets/BS/BSS138.pdf" H 7850 4850 50  0001 L CNN
 	1    7850 4850
@@
 	7650 4950 7650 4850
 $Comp
-L power:+3.3V #PWR?
+L power:+3.3V #PWR037
 U 1 1 5BABDCF1
 P 7250 5200
-F 0 "#PWR?" H 7250 5050 50  0001 C CNN
+F 0 "#PWR037" H 7250 5050 50  0001 C CNN
 F 1 "+3.3V" H 7265 5373 50  0000 C CNN
 F 2 "" H 7250 5200 50  0001 C CNN
@@
 $EndComp
 $Comp
-L power:VCC #PWR?
+L power:VCC #PWR036
 U 1 1 5BABDCF7
 P 7250 4550
-F 0 "#PWR?" H 7250 4400 50  0001 C CNN
+F 0 "#PWR036" H 7250 4400 50  0001 C CNN
 F 1 "VCC" H 7268 4723 50  0000 C CNN
 F 2 "" H 7250 4550 50  0001 C CNN

Commit message: continue on pcb
Parts:
- added U7, U8: HC-SR04, Connector_PinHeader_2.54mm:PinHeader_1x04_P2.54mm_Vertical, symbol localization-symbols:HC-SR04
- R10, R11, R12, R13, R6, R7, R8, R9: footprint Resistor_SMD:R_0603_1608Metric_Pad1.05x0.95mm_HandSolder -> Resistor_SMD:R_1206_3216Metric_Pad1.42x1.75mm_HandSolder
Connections:
- wire segments 52 -> 64
