File: pcb/pcb.sch (KiCad schematic (older format))
At the start: 7 parts

Commit message: Change clock pin
Connections:
- wire segments 77 -> 76
Changed lines of the file:
@@
 EESchema Schematic File Version 4
+LIBS:pcb-cache
 EELAYER 26 0
 EELAYER END
@@
 L Device:Crystal_GND23 Y?
 U 1 1 5BA4C88D
-P 1900 4400
-F 0 "Y?" H 2100 4500 50  0000 L CNN
-F 1 "Crystal_GND23" H 2100 4300 50  0000 L CNN
-F 2 "" H 1900 4400 50  0001 C CNN
-F 3 "~" H 1900 4400 50  0001 C CNN
-	1    1900 4400
+P 1900 5400
+F 0 "Y?" H 2100 5500 50  0000 L CNN
+F 1 "Crystal_GND23" H 2100 5300 50  0000 L CNN
+F 2 "" H 1900 5400 50  0001 C CNN
+F 3 "~" H 1900 5400 50  0001 C CNN
+	1    1900 5400
 	1    0    0    -1
 $EndComp
@@
 L power:GND #PWR?
 U 1 1 5BA4DFE4
-P 1900 4100
-F 0 "#PWR?" H 1900 3850 50  0001 C CNN
-F 1 "GND" H 1905 3927 50  0000 C CNN
-F 2 "" H 1900 4100 50  0001 C CNN
-F 3 "" H 1900 4100 50  0001 C CNN
-	1    1900 4100
+P 1900 5100
+F 0 "#PWR?" H 1900 4850 50  0001 C CNN
+F 1 "GND" H 1905 4927 50  0000 C CNN
+F 2 "" H 1900 5100 50  0001 C CNN
+F 3 "" H 1900 5100 50  0001 C CNN
+	1    1900 5100
 	-1   0    0    1
 $EndComp
 Wire Wire Line
-	1900 4100 1900 4200
+	1900 5100 1900 5200
 $Comp
 L power:+3.3V #PWR?
 U 1 1 5BA4F721
-P 2150 4400
-F 0 "#PWR?" H 2150 4250 50  0001 C CNN
-F 1 "+3.3V" V 2165 4528 50  0000 L CNN
-F 2 "" H 2150 4400 50  0001 C CNN
-F 3 "" H 2150 4400 50  0001 C CNN
-	1    2150 4400
-	0    1    1    0
-$EndComp
-Wire Wire Line
-	2050 4400 2150 4400
+P 2150 5400
+F 0 "#PWR?" H 2150 5250 50  0001 C CNN
+F 1 "+3.3V" V 2165 5528 50  0000 L CNN
+F 2 "" H 2150 5400 50  0001 C CNN
+F 3 "" H 2150 5400 50  0001 C CNN
+	1    2150 5400
+	0    1    1    0
+$EndComp
+Wire Wire Line
+	2050 5400 2150 5400
 $Comp
 L power:+3.3V #PWR?
 U 1 1 5BA50D16
-P 1650 4400
-F 0 "#PWR?" H 1650 4250 50  0001 C CNN
-F 1 "+3.3V" V 1665 4528 50  0000 L CNN
-F 2 "" H 1650 4400 50  0001 C CNN
-F 3 "" H 1650 4400 50  0001 C CNN
-	1    1650 4400
-	0    -1   -1   0
-$EndComp
-Wire Wire Line
-	1650 4400 1750 4400
-Wire Wire Line
-	1900 4600 2850 4600
-Wire Wire Line
-	2850 4600 2850 4000
-Wire Wire Line
-	2850 4000 3050 4000
+P 1650 5400
+F 0 "#PWR?" H 1650 5250 50  0001 C CNN
+F 1 "+3.3V" V 1665 5528 50  0000 L CNN
+F 2 "" H 1650 5400 50  0001 C CNN
+F 3 "" H 1650 5400 50  0001 C CNN
+	1    1650 5400
+	0    -1   -1   0
+$EndComp
+Wire Wire Line
+	1650 5400 1750 5400
 $Comp
 L Connector:Conn_01x07_Female J?
@@
 Wire Wire Line
 	2850 2200 3050 2200
+Wire Wire Line
+	1900 5600 1900 5800
+Wire Wire Line
+	1900 5800 3050 5800
 $EndSCHEMATC

Commit message: Add pcb decoupling
Connections:
- net labels added: VCC_DEC, VSS_DEC
- wire segments 76 -> 86
Changed lines of the file:
@@
 $Descr A4 11693 8268
 encoding utf-8
-Sheet 1 2
+Sheet 1 3
 Title ""
 Date ""
@@
 Wire Wire Line
 	1900 5800 3050 5800
+Wire Wire Line
+	2900 2300 3050 2300
+Wire Wire Line
+	2900 3200 3050 3200
+Wire Wire Line
+	2900 4600 3050 4600
+Wire Wire Line
+	2900 5900 3050 5900
+Text GLabel 2900 2300 0    50   Input ~ 0
+VCC_DEC
+Text GLabel 2900 3200 0    50   Input ~ 0
+VCC_DEC
+Text GLabel 2900 4600 0    50   Input ~ 0
+VCC_DEC
+Text GLabel 2900 5900 0    50   Input ~ 0
+VCC_DEC
+Text GLabel 5400 5900 2    50   Input ~ 0
+VCC_DEC
+Wire Wire Line
+	5250 5900 5400 5900
+Text GLabel 5350 3400 2    50   Input ~ 0
+VCC_DEC
+Wire Wire Line
+	5250 3400 5350 3400
+Text GLabel 2900 3100 0    50   Input ~ 0
+VSS_DEC
+Wire Wire Line
+	2900 3100 3050 3100
+Text GLabel 2900 4700 0    50   Input ~ 0
+VSS_DEC
+Wire Wire Line
+	2900 4700 3050 4700
+Text GLabel 5400 5800 2    50   Input ~ 0
+VSS_DEC
+Wire Wire Line
+	5400 5800 5250 5800
+Text GLabel 5350 3300 2    50   Input ~ 0
+VSS_DEC
+Wire Wire Line
+	5350 3300 5250 3300
+$Sheet
+S 5950 1050 600  300
+U 5BA5978A
+F0 "decoupling" 50
+F1 "decoupling.sch" 50
+$EndSheet
 $EndSCHEMATC

Commit message: lagt til SPI
Parts:
- added J3: Conn_02x03_Counter_Clockwise, symbol Connector_Generic:Conn_02x03_Counter_Clockwise
- added J?: Conn_01x06_Female, symbol Connector:Conn_01x06_Female
- added J?: Conn_01x08_Female, symbol Connector:Conn_01x08_Female
- gave numbers to parts that had none: 7
Connections:
- net labels added: VDD_DEC
- wire segments 86 -> 117
Other:
- note added: "Generic I/O"
- note added: "SPI"
Changed lines of the file:
@@
 $EndDescr
 $Comp
-L localization-symbols:ARDUINO_PYNQ_SHIELD U?
+L localization-symbols:ARDUINO_PYNQ_SHIELD U4
 U 1 1 5BA0F7CD
 P 8550 3450
-F 0 "U?" H 8550 5547 60  0000 C CNN
+F 0 "U4" H 8550 5547 60  0000 C CNN
 F 1 "ARDUINO_PYNQ_SHIELD" H 8550 5441 60  0000 C CNN
 F 2 "" H 9400 2700 60  0001 C CNN
@@
 $EndComp
 $Comp
-L efm32-symbols:EFM32GG980 U?
+L efm32-symbols:EFM32GG980 U1
 U 1 1 5BA3611F
 P 3050 1600
-F 0 "U?" H 4150 1987 60  0000 C CNN
+F 0 "U1" H 4150 1987 60  0000 C CNN
 F 1 "EFM32GG980" H 4150 1881 60  0000 C CNN
 F 2 "QFP100_14X14" H 4150 1840 60  0001 C CNN
@@
 	9800 3300 9600 3300
 $Comp
-L localization-symbols:lidar U?
+L localization-symbols:lidar U3
 U 1 1 5BA3672C
 P 6350 6200
-F 0 "U?" V 6449 6728 50  0000 L CNN
+F 0 "U3" V 6449 6728 50  0000 L CNN
 F 1 "lidar" V 6540 6728 50  0000 L CNN
 F 2 "" H 6350 6200 50  0001 C CNN
@@
 	5250 6600 5250 6500
 $Comp
-L power:+3.3V #PWR?
+L power:+3.3V #PWR0101
 U 1 1 5BA374D8
 P 7350 2900
-F 0 "#PWR?" H 7350 2750 50  0001 C CNN
+F 0 "#PWR0101" H 7350 2750 50  0001 C CNN
 F 1 "+3.3V" V 7365 3028 50  0000 L CNN
 F 2 "" H 7350 2900 50  0001 C CNN
@@
 $EndComp
 $Comp
-L power:VCC #PWR?
+L power:VCC #PWR0102
 U 1 1 5BA3754B
 P 7350 3000
-F 0 "#PWR?" H 7350 2850 50  0001 C CNN
+F 0 "#PWR0102" H 7350 2850 50  0001 C CNN
 F 1 "VCC" V 7368 3127 50  0000 L CNN
 F 2 "" H 7350 3000 50  0001 C CNN
@@
 $EndComp
 $Comp
-L power:GND #PWR?
+L power:GND #PWR0103
 U 1 1 5BA375C1
 P 7350 3100
-F 0 "#PWR?" H 7350 2850 50  0001 C CNN
+F 0 "#PWR0103" H 7350 2850 50  0001 C CNN
 F 1 "GND" V 7355 2972 50  0000 R CNN
 F 2 "" H 7350 3100 50  0001 C CNN
@@
 $EndComp
 $Comp
-L power:GND #PWR?
+L power:GND #PWR0104
 U 1 1 5BA375EF
 P 7350 3200
-F 0 "#PWR?" H 7350 2950 50  0001 C CNN
+F 0 "#PWR0104" H 7350 2950 50  0001 C CNN
 F 1 "GND" V 7355 3072 50  0000 R CNN
 F 2 "" H 7350 3200 50  0001 C CNN
@@
 	7350 3200 7500 3200
 $Comp
-L power:VCC #PWR?
+L power:VCC #PWR0105
 U 1 1 5BA37BF5
 P 6150 6500
-F 0 "#PWR?" H 6150 6350 50  0001 C CNN
+F 0 "#PWR0105" H 6150 6350 50  0001 C CNN
 F 1 "VCC" V 6168 6627 50  0000 L CNN
 F 2 "" H 6150 6500 50  0001 C CNN
@@
 	6150 6500 6250 6500
 $Comp
-L power:VCC #PWR?
+L power:VCC #PWR0106
 U 1 1 5BA37E3E
 P 6150 6100
-F 0 "#PWR?" H 6150 5950 50  0001 C CNN
+F 0 "#PWR0106" H 6150 5950 50  0001 C CNN
 F 1 "VCC" V 6168 6227 50  0000 L CNN
 F 2 "" H 6150 6100 50  0001 C CNN
@@
 	6150 6100 6250 6100
 $Comp
-L power:GND #PWR?
+L power:GND #PWR0107
 U 1 1 5BA380CB
 P 6150 6000
-F 0 "#PWR?" H 6150 5750 50  0001 C CNN
+F 0 "#PWR0107" H 6150 5750 50  0001 C CNN
 F 1 "GND" V 6155 5872 50  0000 R CNN
 F 2 "" H 6150 6000 50  0001 C CNN
@@
 	6150 6000 6250 6000
 $Comp
-L power:GND #PWR?
+L power:GND #PWR0108
 U 1 1 5BA383B0
 P 6150 6700
-F 0 "#PWR?" H 6150 6450 50  0001 C CNN
+F 0 "#PWR0108" H 6150 6450 50  0001 C CNN
 F 1 "GND" V 6155 6572 50  0000 R CNN
 F 2 "" H 6150 6700 50  0001 C CNN
@@
 	6150 6700 6250 6700
 $Comp
-L localization-symbols:IMU U?
+L localization-symbols:IMU U2
 U 1 1 5BA38928
 P 4650 7250
-F 0 "U?" V 4671 6922 50  0000 R CNN
+F 0 "U2" V 4671 6922 50  0000 R CNN
 F 1 "IMU" V 4580 6922 50  0000 R CNN
 F 2 "" V 4800 7150 50  0001 C CNN
@@
 	5500 6200 5250 6200
 $Comp
-L power:VCC #PWR?
+L power:VCC #PWR0109
 U 1 1 5BA39C3E
 P 4900 6900
-F 0 "#PWR?" H 4900 6750 50  0001 C CNN
+F 0 "#PWR0109" H 4900 6750 50  0001 C CNN
 F 1 "VCC" H 4917 7073 50  0000 C CNN
 F 2 "" H 4900 6900 50  0001 C CNN
@@
 	4900 6900 4900 6950
 $Comp
-L power:GND #PWR?
+L power:GND #PWR0110
 U 1 1 5BA3A317
 P 4700 6900
-F 0 "#PWR?" H 4700 6650 50  0001 C CNN
+F 0 "#PWR0110" H 4700 6650 50  0001 C CNN
 F 1 "GND" H 4705 6727 50  0000 C CNN
 F 2 "" H 4700 6900 50  0001 C CNN
@@
 	4500 6750 4500 6950
 $Comp
-L Connector_Generic:Conn_02x10_Odd_Even J?
+L Connector_Generic:Conn_02x10_Odd_Even J2
 U 1 1 5BA3C754
 P 6200 2900
-F 0 "J?" H 6250 3517 50  0000 C CNN
+F 0 "J2" H 6250 3517 50  0000 C CNN
 F 1 "Conn_02x10_Odd_Even" H 6250 3426 50  0000 C CNN
 F 2 "" H 6200 2900 50  0001 C CNN
@@
 Connection ~ 6500 3400
 $Comp
-L power:GND #PWR?
+L power:GND #PWR0111
 U 1 1 5BA3F2DA
 P 6500 3550
-F 0 "#PWR?" H 6500 3300 50  0001 C CNN
+F 0 "#PWR0111" H 6500 3300 50  0001 C CNN
 F 1 "GND" H 6505 3377 50  0000 C CNN
 F 2 "" H 6500 3550 50  0001 C CNN
@@
 	2700 2800 3050 2800
 $Comp
-L Device:Crystal_GND23 Y?
+L Device:Crystal_GND23 Y1
 U 1 1 5BA4C88D
 P 1900 5400
-F 0 "Y?" H 2100 5500 50  0000 L CNN
+F 0 "Y1" H 2100 5500 50  0000 L CNN
 F 1 "Crystal_GND23" H 2100 5300 50  0000 L CNN
 F 2 "" H 1900 5400 50  0001 C CNN
@@
 $EndComp
 $Comp
-L power:GND #PWR?
+L power:GND #PWR0112
 U 1 1 5BA4DFE4
 P 1900 5100
-F 0 "#PWR?" H 1900 4850 50  0001 C CNN
+F 0 "#PWR0112" H 1900 4850 50  0001 C CNN
 F 1 "GND" H 1905 4927 50  0000 C CNN
 F 2 "" H 1900 5100 50  0001 C CNN
@@
 	1900 5100 1900 5200
 $Comp
-L power:+3.3V #PWR?
+L power:+3.3V #PWR0113
 U 1 1 5BA4F721
 P 2150 5400
-F 0 "#PWR?" H 2150 5250 50  0001 C CNN
+F 0 "#PWR0113" H 2150 5250 50  0001 C CNN
 F 1 "+3.3V" V 2165 5528 50  0000 L CNN
 F 2 "" H 2150 5400 50  0001 C CNN
@@
 	2050 5400 2150 5400
 $Comp
-L power:+3.3V #PWR?
+L power:+3.3V #PWR0114
 U 1 1 5BA50D16
 P 1650 5400
-F 0 "#PWR?" H 1650 5250 50  0001 C CNN
+F 0 "#PWR0114" H 1650 5250 50  0001 C CNN
 F 1 "+3.3V" V 1665 5528 50  0000 L CNN
 F 2 "" H 1650 5400 50  0001 C CNN
@@
 	1650 5400 1750 5400
 $Comp
-L Connector:Conn_01x07_Female J?
+L Connector:Conn_01x07_Female J1
 U 1 1 5BA59AD4
 P 2650 1900
-F 0 "J?" H 2544 1375 50  0000 C CNN
+F 0 "J1" H 2544 1375 50  0000 C CNN
 F 1 "Conn_01x07_Female" H 2544 1466 50  0000 C CNN
 F 2 "" H 2650 1900 50  0001 C CNN
@@
 F0 "decoupling" 50
 F1 "decoupling.sch" 50
+F2 "VDD_DEC" I L 5950 1150 50
+F3 "VSS_DEC" I L 5950 1250 50
 $EndSheet
+Text Notes 6500 4800 0    50   ~ 0
+SPI
+$Comp
+L Connector_Generic:Conn_02x03_Counter_Clockwise J3
+U 1 1 5BAC3B31
+P 6200 4800
+F 0 "J3" V 6204 4980 50  0000 L CNN
+F 1 "Conn_02x03_Counter_Clockwise" V 6295 4980 50  0000 L CNN
+F 2 "" H 6200 4800 50  0001 C CNN
+F 3 "~" H 6200 4800 50  0001 C CNN
+	1    6200 4800
+	0    1    1    0
+$EndComp
+Wire Wire Line
+	6300 4600 6300 4500
+Wire Wire Line
+	6300 4500 5550 4500
+Wire Wire Line
+	5550 4500 5550 5000
+Wire Wire Line
+	5550 5000 5250 5000
+Wire Wire Line
+	6200 4600 6200 4550
+Wire Wire Line
+	6200 4550 5600 4550
+Wire Wire Line
+	5600 4550 5600 5100
+Wire Wire Line
+	5600 5100 5250 5100
+Wire Wire Line
+	6200 5100 6200 5200
+Wire Wire Line
+	6200 5200 5750 5200
+Wire Wire Line
+	5750 5200 5750 4900
+Wire Wire Line
+	5750 4900 5250 4900
+Wire Wire Line
+	6100 4600 5650 4600
+Wire Wire Line
+	5650 4600 5650 5200
+Wire Wire Line
+	5650 5200 5250 5200
+Text GLabel 5650 1150 0    50   Input ~ 0
+VDD_DEC
+Text GLabel 5650 1250 0    50   Input ~ 0
+VSS_DEC
+Wire Wire Line
+	5950 1150 5650 1150
+Wire Wire Line
+	5950 1250 5650 1250
+$Comp
+L Connector:Conn_01x06_Female J?
+U 1 1 5BB2F41D
+P 1900 6300
+F 0 "J?" H 1794 5775 50  0000 C CNN
+F 1 "Conn_01x06_Female" H 1794 5866 50  0000 C CNN
+F 2 "" H 1900 6300 50  0001 C CNN
+F 3 "~" H 1900 6300 50  0001 C CNN
+	1    1900 6300
+	-1   0    0    1
+$EndComp
+Wire Wire Line
+	3050 6500 2100 6500
+Wire Wire Line
+	2100 6400 3050 6400
+Wire Wire Line
+	3050 6300 2100 6300
+Wire Wire Line
+	2100 6200 3050 6200
+Wire Wire Line
+	3050 6100 2100 6100
+Wire Wire Line
+	2100 6000 3050 6000
+Text Notes 1300 6100 0    50   ~ 0
+Generic I/O
+$Comp
+L Connector:Conn_01x08_Female J?
+U 1 1 5BB45AA7
+P 7000 1900
+F 0 "J?" H 7027 1876 50  0000 L CNN
+F 1 "Conn_01x08_Female" H 7027 1785 50  0000 L CNN
+F 2 "" H 7000 1900 50  0001 C CNN
+F 3 "~" H 7000 1900 50  0001 C CNN
+	1    7000 1900
+	1    0    0    -1
+$EndComp
+Wire Wire Line
+	6800 1600 5250 1600
+Wire Wire Line
+	5250 1700 6800 1700
+Wire Wire Line
+	6800 1800 5250 1800
+Wire Wire Line
+	5250 1900 6800 1900
+Wire Wire Line
+	6800 2000 5250 2000
+Wire Wire Line
+	5250 2100 6800 2100
+Wire Wire Line
+	6800 2200 5250 2200
+Wire Wire Line
+	5250 2300 6800 2300
+Text Notes 7150 1750 0    50   ~ 0
+Generic I/O
 $EndSCHEMATC

Commit message: Added levelswitch
Parts:
- added J?: Conn_01x04_Male, symbol Connector:Conn_01x04_Male
Connections:
- net labels added: +5V
- wire segments 117 -> 121
Other:
- note added: "Debug pynq\n"
- note added: "debug EFM"
Changed lines of the file:
@@
 $Descr A4 11693 8268
 encoding utf-8
-Sheet 1 3
+Sheet 1 4
 Title ""
 Date ""
@@
 F2 "LED_1" I R 2200 2500 50
 F3 "LED_2" I R 2200 2600 50
-F4 "LED_3" I R 2200 2700 50
-F5 "LED_4" I R 2200 2800 50
-F6 "SW_1" I R 2200 3250 50
-F7 "SW_2" I R 2200 3350 50
+F4 "LED_3" I R 2200 3250 50
+F5 "LED_4" I R 2200 3350 50
+F6 "SW_1" I R 2200 2700 50
+F7 "SW_2" I R 2200 2800 50
 F8 "SW_3" I R 2200 3450 50
 F9 "SW_4" I R 2200 3550 50
@@
 Wire Wire Line
 	2200 2600 3050 2600
-Wire Wire Line
-	2200 3250 2650 3250
-Wire Wire Line
-	2650 3250 2650 2700
-Wire Wire Line
-	2650 2700 3050 2700
-Wire Wire Line
-	2200 3350 2700 3350
-Wire Wire Line
-	2700 3350 2700 2800
-Wire Wire Line
-	2700 2800 3050 2800
 $Comp
 L Device:Crystal_GND23 Y1
@@
 $EndComp
 Wire Wire Line
-	3050 6500 2100 6500
-Wire Wire Line
-	2100 6400 3050 6400
-Wire Wire Line
 	3050 6300 2100 6300
 Wire Wire Line
@@
 Text Notes 7150 1750 0    50   ~ 0
 Generic I/O
+$Sheet
+S 2300 6300 550  700
+U 5BAA6CA9
+F0 "levelswitch" 50
+F1 "levelswitch.sch" 50
+F2 "LV" I R 2850 6800 50
+F3 "HV" I R 2850 6900 50
+F4 "GND" I L 2300 6900 50
+F5 "LV1" I R 2850 6400 50
+F6 "LV2" I R 2850 6500 50
+F7 "HV1" I L 2300 6400 50
+F8 "HV2" I L 2300 6500 50
+$EndSheet
+Wire Wire Line
+	3050 6400 2850 6400
+Wire Wire Line
+	2850 6500 3050 6500
+Wire Wire Line
+	2300 6400 2100 6400
+Wire Wire Line
+	2100 6500 2300 6500
+Wire Wire Line
+	2200 2700 3050 2700
+Wire Wire Line
+	2200 2800 3050 2800
+$Comp
+L Connector:Conn_01x04_Male J?
+U 1 1 5BAE10AA
+P 2500 3450
+F 0 "J?" H 2473 3330 50  0000 R CNN
+F 1 "Conn_01x04_Male" H 2473 3421 50  0000 R CNN
+F 2 "" H 2500 3450 50  0001 C CNN
+F 3 "~" H 2500 3450 50  0001 C CNN
+	1    2500 3450
+	-1   0    0    1
+$EndComp
+Wire Wire Line
+	2300 3250 2200 3250
+Wire Wire Line
+	2300 3350 2200 3350
+Wire Wire Line
+	2300 3450 2200 3450
+Wire Wire Line
+	2300 3550 2200 3550
+Text Notes 2400 3700 0    50   ~ 0
+Debug pynq\n
+Text Notes 2300 2400 0    50   ~ 0
+debug EFM
+$Comp
+L power:+3.3V #PWR?
+U 1 1 5BAF583C
+P 3350 6800
+F 0 "#PWR?" H 3350 6650 50  0001 C CNN
+F 1 "+3.3V" V 3365 6928 50  0000 L CNN
+F 2 "" H 3350 6800 50  0001 C CNN
+F 3 "" H 3350 6800 50  0001 C CNN
+	1    3350 6800
+	0    1    1    0
+$EndComp
+$Comp
+L power:+5V #PWR?
+U 1 1 5BAF58B4
+P 3500 6900
+F 0 "#PWR?" H 3500 6750 50  0001 C CNN
+F 1 "+5V" V 3515 7028 50  0000 L CNN
+F 2 "" H 3500 6900 50  0001 C CNN
+F 3 "" H 3500 6900 50  0001 C CNN
+	1    3500 6900
+	0    1    1    0
+$EndComp
+Wire Wire Line
+	3350 6800 2850 6800
+Wire Wire Line
+	3500 6900 2850 6900
 $EndSCHEMATC

Commit message: Prettyfy Schematic
Parts:
- removed J1: Conn_01x07_Female, symbol Connector:Conn_01x07_Female
- removed J2: Conn_02x10_Odd_Even, symbol Connector_Generic:Conn_02x10_Odd_Even
- removed J3: Conn_02x03_Counter_Clockwise, symbol Connector_Generic:Conn_02x03_Counter_Clockwise
- removed J?: Conn_01x04_Male, symbol Connector:Conn_01x04_Male
- removed J?: Conn_01x06_Female, symbol Connector:Conn_01x06_Female
- removed J?: Conn_01x08_Female, symbol Connector:Conn_01x08_Female
- removed U2: IMU, symbol localization-symbols:IMU
- removed U3: lidar, symbol localization-symbols:lidar
- removed Y1: Crystal_GND23, symbol Device:Crystal_GND23
- U1: footprint QFP100_14X14 -> efm32-footprints:EFM32GG980
- renumbered U4 to U2
Connections:
- net labels added: AVDD_DEC, DEC, IOVDD_DEC, MCU_RST, PYNQ_RX, PYNQ_SCL, PYNQ_SDA, PYNQ_TX
- net labels removed: EFM32_RST, VCC_DEC, VDD_DEC
- wire segments 121 -> 39
Other:
- note removed: "Debug pynq\n"
- note removed: "Generic I/O"
- note removed: "SPI"
- note removed: "debug EFM"

Commit message: Add PYNQ debug pins
Parts:
- added JP? (x4): M08, symbol DMPro17-rescue:M08
- added JP?: M10, symbol DMPro17-rescue:M10
- added JP? (x2): M06, symbol DMPro17-rescue:M06
- added JP?: M04, symbol DMPro17-rescue:M04
Connections:
- net labels removed: +5V
- wire segments 39 -> 105

Commit message: Finishe schematic, add netlist and start editing pcb design
Parts:
- added JP1: M06, Connector_PinHeader_2.54mm:PinHeader_1x06_P2.54mm_Vertical, symbol freetronics_schematic:M06
- JP2, JP3, JP4, JP9: renamed from JP?; footprint (none) -> Connector_PinHeader_2.54mm:PinHeader_1x08_P2.54mm_Vertical
- JP5: renamed from JP?; footprint (none) -> Connector_PinHeader_2.54mm:PinHeader_1x10_P2.54mm_Vertical
- JP6, JP8: renamed from JP?; footprint (none) -> Connector_PinHeader_2.54mm:PinHeader_1x06_P2.54mm_Vertical
- JP7: renamed from JP?; footprint (none) -> Connector_PinHeader_2.54mm:PinHeader_1x04_P2.54mm_Vertical
- U2: footprint (none) -> localization-footprints:ARDUINO_PYNQ_SHIELD
Connections:
- wire segments 105 -> 123
Changed lines of the file:
@@
 	5250 6600 5250 6500
 $Sheet
-S 2100 2400 600  500
+S 2100 1500 600  500
 U 5BA41DB8
 F0 "EFM_DEBUG" 50
 F1 "EFM_DEBUG.sch" 50
-F2 "LED_1" I R 2700 2500 50
-F3 "LED_2" I R 2700 2600 50
-F4 "SW_1" I R 2700 2700 50
-F5 "SW_2" I R 2700 2800 50
+F2 "LED_1" I R 2700 1600 50
+F3 "LED_2" I R 2700 1700 50
+F4 "SW_1" I R 2700 1800 50
+F5 "SW_2" I R 2700 1900 50
 $EndSheet
 $Sheet
@@
 Wire Wire Line
 	6100 6400 6250 6400
-Wire Wire Line
-	2700 2500 3050 2500
-Wire Wire Line
-	2700 2600 3050 2600
-Wire Wire Line
-	2700 2700 3050 2700
-Wire Wire Line
-	2700 2800 3050 2800
 Text Label 5250 5900 0    50   ~ 0
 IOVDD_DEC
@@
 F 0 "U2" H 9100 5797 60  0000 C CNN
 F 1 "ARDUINO_PYNQ_SHIELD" H 9100 5691 60  0000 C CNN
-F 2 "" H 9950 2950 60  0001 C CNN
+F 2 "localization-footprints:ARDUINO_PYNQ_SHIELD" H 9950 2950 60  0001 C CNN
 F 3 "" H 9950 2950 60  0001 C CNN
 	1    9100 3700
@@
 	2500 4400 3050 4400
 $Comp
-L DMPro17-rescue:M08 JP?
+L DMPro17-rescue:M08 JP2
 U 1 1 5BAC634F
 P 7650 2650
-F 0 "JP?" H 7469 1729 50  0000 C CNN
+F 0 "JP2" H 7469 1729 50  0000 C CNN
 F 1 "M08" H 7469 1813 40  0000 C CNN
-F 2 "" H 7650 2650 60  0000 C CNN
+F 2 "Connector_PinHeader_2.54mm:PinHeader_1x08_P2.54mm_Vertical" H 7650 2650 60  0001 C CNN
 F 3 "" H 7650 2650 60  0000 C CNN
 	1    7650 2650
@@
 $EndComp
 $Comp
-L DMPro17-rescue:M08 JP?
+L DMPro17-rescue:M08 JP3
 U 1 1 5BAC63E8
 P 7650 3550
-F 0 "JP?" H 7469 2629 50  0000 C CNN
+F 0 "JP3" H 7469 2629 50  0000 C CNN
 F 1 "M08" H 7469 2713 40  0000 C CNN
-F 2 "" H 7650 3550 60  0000 C CNN
+F 2 "Connector_PinHeader_2.54mm:PinHeader_1x08_P2.54mm_Vertical" H 7650 3550 60  0001 C CNN
 F 3 "" H 7650 3550 60  0000 C CNN
 	1    7650 3550
@@
 $EndComp
 $Comp
-L DMPro17-rescue:M08 JP?
+L DMPro17-rescue:M08 JP4
 U 1 1 5BAC647C
 P 7650 4450
-F 0 "JP?" H 7469 3529 50  0000 C CNN
+F 0 "JP4" H 7469 3529 50  0000 C CNN
 F 1 "M08" H 7469 3613 40  0000 C CNN
-F 2 "" H 7650 4450 60  0000 C CNN
+F 2 "Connector_PinHeader_2.54mm:PinHeader_1x08_P2.54mm_Vertical" H 7650 4450 60  0001 C CNN
 F 3 "" H 7650 4450 60  0000 C CNN
 	1    7650 4450
@@
 	8050 4450 7950 4450
 $Comp
-L DMPro17-rescue:M10 JP?
+L DMPro17-rescue:M10 JP5
 U 1 1 5BAE89E7
 P 7650 5550
-F 0 "JP?" H 7469 4429 50  0000 C CNN
+F 0 "JP5" H 7469 4429 50  0000 C CNN
 F 1 "M10" H 7469 4513 40  0000 C CNN
-F 2 "" H 7650 5550 60  0000 C CNN
+F 2 "Connector_PinHeader_2.54mm:PinHeader_1x10_P2.54mm_Vertical" H 7650 5550 60  0001 C CNN
 F 3 "" H 7650 5550 60  0000 C CNN
 	1    7650 5550
@@
 Connection ~ 7950 5550
 $Comp
-L DMPro17-rescue:M06 JP?
+L DMPro17-rescue:M06 JP6
 U 1 1 5BB0CADE
 P 10600 1950
-F 0 "JP?" H 10578 1728 50  0000 L CNN
+F 0 "JP6" H 10578 1728 50  0000 L CNN
 F 1 "M06" H 10578 1644 40  0000 L CNN
-F 2 "" H 10600 1950 60  0000 C CNN
+F 2 "Connector_PinHeader_2.54mm:PinHeader_1x06_P2.54mm_Vertical" H 10600 1950 60  0001 C CNN
 F 3 "" H 10600 1950 60  0000 C CNN
 	1    10600 1950
@@
 	10150 2450 10300 2450
 $Comp
-L DMPro17-rescue:M04 JP?
+L DMPro17-rescue:M04 JP7
 U 1 1 5BB1CAA8
 P 10600 2650
-F 0 "JP?" H 10578 2528 50  0000 L CNN
+F 0 "JP7" H 10578 2528 50  0000 L CNN
 F 1 "M04" H 10578 2444 40  0000 L CNN
-F 2 "" H 10600 2650 60  0000 C CNN
+F 2 "Connector_PinHeader_2.54mm:PinHeader_1x04_P2.54mm_Vertical" H 10600 2650 60  0001 C CNN
 F 3 "" H 10600 2650 60  0000 C CNN
 	1    10600 2650
@@
 	10150 2950 10300 2950
 $Comp
-L DMPro17-rescue:M06 JP?
+L DMPro17-rescue:M06 JP8
 U 1 1 5BB28935
 P 10600 3150
-F 0 "JP?" H 10578 2928 50  0000 L CNN
+F 0 "JP8" H 10578 2928 50  0000 L CNN
 F 1 "M06" H 10578 2844 40  0000 L CNN
-F 2 "" H 10600 3150 60  0000 C CNN
+F 2 "Connector_PinHeader_2.54mm:PinHeader_1x06_P2.54mm_Vertical" H 10600 3150 60  0001 C CNN
 F 3 "" H 10600 3150 60  0000 C CNN
 	1    10600 3150
@@
 	10150 3650 10300 3650
 $Comp
-L DMPro17-rescue:M08 JP?
+L DMPro17-rescue:M08 JP9
 U 1 1 5BB3FDEB
 P 10600 3850
-F 0 "JP?" H 10578 3528 50  0000 L CNN
+F 0 "JP9" H 10578 3528 50  0000 L CNN
 F 1 "M08" H 10578 3444 40  0000 L CNN
-F 2 "" H 10600 3850 60  0000 C CNN
+F 2 "Connector_PinHeader_2.54mm:PinHeader_1x08_P2.54mm_Vertical" H 10600 3850 60  0001 C CNN
 F 3 "" H 10600 3850 60  0000 C CNN
 	1    10600 3850
@@
 Wire Wire Line
 	7400 4250 7950 4250
+Wire Wire Line
+	5250 2400 7650 2400
+Wire Wire Line
+	7650 2400 7650 2350
+Wire Wire Line
+	7650 2350 7950 2350
+Connection ~ 7950 2350
+Wire Wire Line
+	5250 2500 7650 2500
+Wire Wire Line
+	7650 2500 7650 2450
+Wire Wire Line
+	7650 2450 7950 2450
+Connection ~ 7950 2450
+Wire Wire Line
+	5250 2600 7650 2600
+Wire Wire Line
+	7650 2600 7650 2550
+Wire Wire Line
+	7650 2550 7950 2550
+Connection ~ 7950 2550
+Wire Wire Line
+	5250 2700 7650 2700
+Wire Wire Line
+	7650 2700 7650 2650
+Wire Wire Line
+	7650 2650 7950 2650
+Connection ~ 7950 2650
+Wire Wire Line
+	2700 1600 3050 1600
+Wire Wire Line
+	2700 1700 3050 1700
+Wire Wire Line
+	3050 1800 2700 1800
+Wire Wire Line
+	2700 1900 3050 1900
+$Comp
+L freetronics_schematic:M06 JP1
+U 1 1 5BB0C3BE
+P 2050 2900
+F 0 "JP1" H 1869 2179 50  0000 C CNN
+F 1 "M06" H 1869 2263 40  0000 C CNN
+F 2 "Connector_PinHeader_2.54mm:PinHeader_1x06_P2.54mm_Vertical" H 2050 2900 60  0001 C CNN
+F 3 "" H 2050 2900 60  0000 C CNN
+	1    2050 2900
+	-1   0    0    1
+$EndComp
+Wire Wire Line
+	2350 2400 3050 2400
+Wire Wire Line
+	3050 2500 2350 2500
+Wire Wire Line
+	2350 2600 3050 2600
+Wire Wire Line
+	3050 2700 2350 2700
+Wire Wire Line
+	2350 2800 3050 2800
+Wire Wire Line
+	3050 2900 2350 2900
 $EndSCHEMATC
