File: pcb/pcb.sch (KiCad schematic (older format))
At the start: 11 parts, among them U1 EFM32GG980, U2 ARDUINO_PYNQ_SHIELD

Commit message: continue on pcb
Parts:
- added J3: Conn_01x03_Female, Connector_PinSocket_2.54mm:PinSocket_1x03_P2.54mm_Vertical, symbol Connector:Conn_01x03_Female
Connections:
- net labels added: +3V3
- wire segments 123 -> 128
Changed lines of the file:
@@
 Wire Wire Line
 	6100 6200 6250 6200
-Wire Wire Line
-	5250 6600 5250 6500
 $Sheet
 S 2100 1500 600  500
@@
 F4 "MOTO_CTRL" I L 6250 6400 50
 $EndSheet
-$Comp
-L efm32-symbols:EFM32GG980 U1
-U 1 1 5BA3611F
-P 3050 1600
-F 0 "U1" H 4150 1987 60  0000 C CNN
-F 1 "EFM32GG980" H 4150 1881 60  0000 C CNN
-F 2 "efm32-footprints:EFM32GG980" H 4150 1840 60  0001 C CNN
-F 3 "" H 3050 1600 60  0000 C CNN
-	1    3050 1600
-	1    0    0    -1
-$EndComp
-Wire Wire Line
-	5250 6600 6100 6600
-Wire Wire Line
-	6100 6600 6100 6400
-Wire Wire Line
-	6100 6400 6250 6400
 Text Label 5250 5900 0    50   ~ 0
 IOVDD_DEC
@@
 $Comp
 L power:VCC #PWR05
-U 1 1 5BB2DED4
+U 1 1 5BB359F6
 P 10650 4150
 F 0 "#PWR05" H 10650 4000 50  0001 C CNN
@@
 Wire Wire Line
 	2700 1700 3050 1700
-Wire Wire Line
-	3050 1800 2700 1800
-Wire Wire Line
-	2700 1900 3050 1900
 $Comp
 L freetronics_schematic:M06 JP1
@@
 Wire Wire Line
 	3050 2900 2350 2900
+$Comp
+L efm32-symbols:EFM32GG980 U1
+U 1 1 5BA3611F
+P 3050 1600
+F 0 "U1" H 4150 1987 60  0000 C CNN
+F 1 "EFM32GG980" H 4150 1881 60  0000 C CNN
+F 2 "efm32-footprints:EFM32GG980" H 4150 1840 60  0001 C CNN
+F 3 "" H 3050 1600 60  0000 C CNN
+	1    3050 1600
+	1    0    0    -1
+$EndComp
+Wire Wire Line
+	6250 6400 5900 6400
+Wire Wire Line
+	5900 6400 5900 4600
+Wire Wire Line
+	5900 4600 5250 4600
+$Comp
+L Connector:Conn_01x03_Female J3
+U 1 1 5BB35F8F
+P 10450 5700
+F 0 "J3" H 10477 5726 50  0000 L CNN
+F 1 "Conn_01x03_Female" H 10477 5635 50  0000 L CNN
+F 2 "Connector_PinSocket_2.54mm:PinSocket_1x03_P2.54mm_Vertical" H 10450 5700 50  0001 C CNN
+F 3 "~" H 10450 5700 50  0001 C CNN
+	1    10450 5700
+	1    0    0    -1
+$EndComp
+$Comp
+L power:VCC #PWR0107
+U 1 1 5BB36082
+P 10250 5600
+F 0 "#PWR0107" H 10250 5450 50  0001 C CNN
+F 1 "VCC" H 10267 5773 50  0000 C CNN
+F 2 "" H 10250 5600 50  0001 C CNN
+F 3 "" H 10250 5600 50  0001 C CNN
+	1    10250 5600
+	1    0    0    -1
+$EndComp
+$Comp
+L power:+3V3 #PWR0108
+U 1 1 5BB36162
+P 10250 5700
+F 0 "#PWR0108" H 10250 5550 50  0001 C CNN
+F 1 "+3V3" V 10265 5828 50  0000 L CNN
+F 2 "" H 10250 5700 50  0001 C CNN
+F 3 "" H 10250 5700 50  0001 C CNN
+	1    10250 5700
+	0    -1   -1   0
+$EndComp
+$Comp
+L power:GND #PWR0109
+U 1 1 5BB3620B
+P 10250 5800
+F 0 "#PWR0109" H 10250 5550 50  0001 C CNN
+F 1 "GND" H 10255 5627 50  0000 C CNN
+F 2 "" H 10250 5800 50  0001 C CNN
+F 3 "" H 10250 5800 50  0001 C CNN
+	1    10250 5800
+	1    0    0    -1
+$EndComp
+Wire Wire Line
+	3050 1900 2800 1900
+Wire Wire Line
+	2800 1900 2800 1800
+Wire Wire Line
+	2800 1800 2700 1800
+Wire Wire Line
+	3050 1800 2950 1800
+Wire Wire Line
+	2950 1800 2950 1950
+Wire Wire Line
+	2950 1950 2750 1950
+Wire Wire Line
+	2750 1950 2750 1900
+Wire Wire Line
+	2750 1900 2700 1900
 $EndSCHEMATC
