File: pcb/pcb.sch (KiCad schematic (older format))
At the start: 10 parts, among them U1 EFM32GG980, U2 ARDUINO_PYNQ_SHIELD

Commit message: Connect some more wires
Connections:
- net labels added: PB11, PB12, PB4, PB5, PC0, PC1, PD5, PD6
- net labels removed: PF6, PF7
- wire segments 108 -> 100
Changed lines of the file:
@@
 $EndDescr
 $Sheet
-S 2100 1500 600  500
+S 5650 4600 600  500
 U 5BA41DB8
 F0 "EFM_DEBUG" 50
 F1 "EFM_DEBUG.sch" 50
-F2 "LED_1" I R 2700 1600 50
-F3 "LED_2" I R 2700 1700 50
-F4 "SW_1" I R 2700 1800 50
-F5 "SW_2" I R 2700 1900 50
+F2 "LED_1" I L 5650 5000 50
+F3 "LED_2" I L 5650 4900 50
+F4 "SW_1" I L 5650 4800 50
+F5 "SW_2" I L 5650 4700 50
 $EndSheet
 $Sheet
@@
 IOVDD_DEC
 $Sheet
-S 6200 4800 550  500
+S 2050 6000 550  500
 U 5BAD9CF1
 F0 "SPI" 50
 F1 "SPI.sch" 50
-F2 "MOSI" I L 6200 4900 50
-F3 "MISO" I L 6200 5000 50
-F4 "SCLK" I L 6200 5100 50
-F5 "SS" I L 6200 5200 50
-$EndSheet
-Wire Wire Line
-	5250 5200 6200 5200
-Wire Wire Line
-	5250 5100 6200 5100
-Wire Wire Line
-	5250 5000 6200 5000
-Wire Wire Line
-	5250 4900 6200 4900
+F2 "MOSI" I R 2600 6100 50
+F3 "MISO" I R 2600 6200 50
+F4 "SCLK" I R 2600 6300 50
+F5 "SS" I R 2600 6400 50
+$EndSheet
 $Sheet
 S 2100 5600 500  150
@@
 	5850 1250 5950 1250
 $Sheet
-S 5300 6150 550  300
+S 2350 3650 550  300
 U 5BB1BAF2
 F0 "IMU" 50
 F1 "IMU.sch" 50
-F2 "RST" I L 5300 6200 50
-F3 "SCL" I L 5300 6300 50
-F4 "SDA" I L 5300 6400 50
-$EndSheet
-Wire Wire Line
-	5250 6200 5300 6200
-Wire Wire Line
-	5250 6300 5300 6300
-Wire Wire Line
-	5250 6400 5300 6400
-$Sheet
-S 6250 6150 500  300
+F2 "RST" I R 2900 3900 50
+F3 "SCL" I R 2900 3800 50
+F4 "SDA" I R 2900 3700 50
+$EndSheet
+$Sheet
+S 5850 2950 500  300
 U 5BB1F7DF
 F0 "LIDAR" 50
 F1 "LIDAR.sch" 50
-F2 "RX" I L 6250 6200 50
-F3 "TX" I L 6250 6300 50
-F4 "MOTO_CTRL" I L 6250 6400 50
+F2 "RX" I L 5850 3100 50
+F3 "TX" I L 5850 3200 50
+F4 "MOTO_CTRL" I L 5850 3000 50
 $EndSheet
 Text Label 5250 5900 0    50   ~ 0
@@
 Text Label 7550 5550 2    50   ~ 0
 PYNQ_SCL
-Text Label 3050 5400 2    50   ~ 0
+Text Label 5250 6100 0    50   ~ 0
 PYNQ_SDA
-Text Label 3050 5500 2    50   ~ 0
+Text Label 5250 6000 0    50   ~ 0
 PYNQ_SCL
 $Sheet
@@
 	7650 2650 7950 2650
 Connection ~ 7950 2650
-Wire Wire Line
-	2700 1600 3050 1600
-Wire Wire Line
-	2700 1700 3050 1700
 $Comp
 L efm32-symbols:EFM32GG980 U1
@@
 	1    0    0    -1
 $EndComp
-Wire Wire Line
-	6250 6400 5900 6400
-Wire Wire Line
-	5900 6400 5900 4600
-Wire Wire Line
-	5900 4600 5250 4600
-Wire Wire Line
-	1650 3400 3050 3400
-Wire Wire Line
-	1650 3700 3050 3700
-Wire Wire Line
-	1650 3800 3050 3800
-Wire Wire Line
-	1650 4100 3050 4100
-Wire Wire Line
-	1650 4200 3050 4200
-Wire Wire Line
-	1650 3300 2600 3300
-Wire Wire Line
-	2600 3300 2600 2800
-Wire Wire Line
-	2600 2800 3050 2800
-Text Label 5250 3200 0    50   ~ 0
-PF6
-Text Label 5250 3100 0    50   ~ 0
-PF7
-Text Label 6250 6300 2    50   ~ 0
-PF6
-Text Label 6250 6200 2    50   ~ 0
-PF7
 Text Label 1650 3600 0    50   ~ 0
 PF10
@@
 Text Label 3050 1900 2    50   ~ 0
 PA3
+Wire Wire Line
+	2600 6100 3050 6100
+Wire Wire Line
+	2600 6200 3050 6200
+Wire Wire Line
+	2600 6300 3050 6300
+Wire Wire Line
+	2600 6400 3050 6400
+Wire Wire Line
+	2900 3700 3050 3700
+Wire Wire Line
+	2900 3800 3050 3800
+Wire Wire Line
+	2900 3900 3050 3900
+Text Label 1650 3300 0    50   ~ 0
+PD5
+Text Label 1650 3400 0    50   ~ 0
+PD6
+Text Label 1650 3700 0    50   ~ 0
+PB11
+Text Label 1650 3800 0    50   ~ 0
+PB12
+Text Label 1650 4100 0    50   ~ 0
+PB4
+Text Label 1650 4200 0    50   ~ 0
+PB5
+Text Label 5250 6500 0    50   ~ 0
+PD5
+Text Label 5250 6400 0    50   ~ 0
+PD6
+Text Label 3050 5400 2    50   ~ 0
+PB11
+Text Label 3050 5500 2    50   ~ 0
+PB12
+Text Label 3050 2800 2    50   ~ 0
+PB4
+Text Label 3050 2900 2    50   ~ 0
+PB5
+Wire Wire Line
+	5850 3200 5250 3200
+Wire Wire Line
+	5250 3100 5850 3100
+Wire Wire Line
+	5850 3000 5250 3000
+Wire Wire Line
+	5650 5000 5250 5000
+Wire Wire Line
+	5650 4900 5250 4900
+Text Label 5650 4700 2    50   ~ 0
+PC0
+Text Label 5650 4800 2    50   ~ 0
+PC1
+Text Label 3050 3300 2    50   ~ 0
+PC0
+Text Label 3050 3400 2    50   ~ 0
+PC1
 $EndSCHEMATC

Commit message: Think it is somewhat finished
Parts:
- renumbered JP2 to JP1, JP3 to JP2, JP4 to JP3, JP5 to JP4, JP6 to JP5, JP7 to JP6, JP8 to JP7, JP9 to JP8
Connections:
- net labels added: PA7_C1, PA8_C2, PA9_IMU_INT, PB10_IMU_RST, PB11_IMU_SDA, PB12_IMU_SCL, PB7_CTX, PB8_CRX, PC0_B1, PC1_B2, PC2_BTX, PC3_BRX, PD6_A1, PD7_A2, PF10_ATX, PF11_ARX
- net labels removed: PA3, PA4, PB10, PB11, PB12, PB4, PB5, PB9, PC0, PC1, PD5, PD6, PF10, PF11
- wire segments 100 -> 91
- no-connect marks 0 -> 1
Changed lines of the file:
@@
 $EndDescr
 $Sheet
-S 5650 4600 600  500
+S 5350 4400 600  500
 U 5BA41DB8
 F0 "EFM_DEBUG" 50
 F1 "EFM_DEBUG.sch" 50
-F2 "LED_1" I L 5650 5000 50
-F3 "LED_2" I L 5650 4900 50
-F4 "SW_1" I L 5650 4800 50
-F5 "SW_2" I L 5650 4700 50
+F2 "LED_1" I L 5350 4800 50
+F3 "LED_2" I L 5350 4700 50
+F4 "SW_1" I L 5350 4500 50
+F5 "SW_2" I L 5350 4600 50
 $EndSheet
 $Sheet
@@
 	5850 1250 5950 1250
 $Sheet
-S 2350 3650 550  300
+S 1400 4550 550  400
 U 5BB1BAF2
 F0 "IMU" 50
 F1 "IMU.sch" 50
-F2 "RST" I R 2900 3900 50
-F3 "SCL" I R 2900 3800 50
-F4 "SDA" I R 2900 3700 50
+F2 "RST" I R 1950 4800 50
+F3 "SCL" I R 1950 4700 50
+F4 "SDA" I R 1950 4600 50
+F5 "INT" I R 1950 4900 50
 $EndSheet
 $Sheet
@@
 $EndComp
 $Comp
-L power:GND #PWR03
+L power:GND #PWR01
 U 1 1 5BB2DDEE
 P 10650 3950
-F 0 "#PWR03" H 10650 3700 50  0001 C CNN
+F 0 "#PWR01" H 10650 3700 50  0001 C CNN
 F 1 "GND" V 10655 3822 50  0000 R CNN
 F 2 "" H 10650 3950 50  0001 C CNN
@@
 $EndComp
 $Comp
-L power:GND #PWR04
+L power:GND #PWR02
 U 1 1 5BB2DE61
 P 10650 4050
-F 0 "#PWR04" H 10650 3800 50  0001 C CNN
+F 0 "#PWR02" H 10650 3800 50  0001 C CNN
 F 1 "GND" V 10655 3922 50  0000 R CNN
 F 2 "" H 10650 4050 50  0001 C CNN
@@
 $EndComp
 $Comp
-L power:VCC #PWR05
+L power:VCC #PWR03
 U 1 1 5BB359F6
 P 10650 4150
-F 0 "#PWR05" H 10650 4000 50  0001 C CNN
+F 0 "#PWR03" H 10650 4000 50  0001 C CNN
 F 1 "VCC" V 10667 4278 50  0000 L CNN
 F 2 "" H 10650 4150 50  0001 C CNN
@@
 $EndComp
 $Comp
-L power:+3.3V #PWR06
+L power:+3.3V #PWR04
 U 1 1 5BB2DF38
 P 10650 4250
-F 0 "#PWR06" H 10650 4100 50  0001 C CNN
+F 0 "#PWR04" H 10650 4100 50  0001 C CNN
 F 1 "+3.3V" V 10665 4378 50  0000 L CNN
 F 2 "" H 10650 4250 50  0001 C CNN
@@
 PYNQ_SCL
 $Sheet
-S 1100 3250 550  1250
+S 1100 1850 550  1250
 U 5BAB97A9
 F0 "SONAR-GPIO" 50
 F1 "SONAR-GPIO.sch" 50
-F2 "AD1" I R 1650 3300 50
-F3 "AD2" I R 1650 3400 50
-F4 "AD3_RX" I R 1650 3500 50
-F5 "AD4_TX" I R 1650 3600 50
-F6 "BD1" I R 1650 3700 50
-F7 "BD2" I R 1650 3800 50
-F8 "BD3_RX" I R 1650 3900 50
-F9 "BD4_TX" I R 1650 4000 50
-F10 "CD1" I R 1650 4100 50
-F11 "CD2" I R 1650 4200 50
-F12 "C3_RX" I R 1650 4300 50
-F13 "CD4_TX" I R 1650 4400 50
-$EndSheet
-$Comp
-L DMPro17-rescue:M08 JP2
+F2 "A1" I R 1650 1900 50
+F3 "A2" I R 1650 2000 50
+F4 "A3" I R 1650 2100 50
+F5 "A4" I R 1650 2200 50
+F6 "B1" I R 1650 2300 50
+F7 "B2" I R 1650 2400 50
+F8 "B3" I R 1650 2500 50
+F9 "B4" I R 1650 2600 50
+F10 "C1" I R 1650 2700 50
+F11 "C2" I R 1650 2800 50
+F12 "C3" I R 1650 2900 50
+F13 "C4" I R 1650 3000 50
+$EndSheet
+$Comp
+L DMPro17-rescue:M08 JP1
 U 1 1 5BAC634F
 P 7650 2650
-F 0 "JP2" H 7469 1729 50  0000 C CNN
+F 0 "JP1" H 7469 1729 50  0000 C CNN
 F 1 "M08" H 7469 1813 40  0000 C CNN
 F 2 "Connector_PinHeader_2.54mm:PinHeader_1x08_P2.54mm_Vertical" H 7650 2650 60  0001 C CNN
@@
 $EndComp
 $Comp
-L DMPro17-rescue:M08 JP3
+L DMPro17-rescue:M08 JP2
 U 1 1 5BAC63E8
 P 7650 3550
-F 0 "JP3" H 7469 2629 50  0000 C CNN
+F 0 "JP2" H 7469 2629 50  0000 C CNN
 F 1 "M08" H 7469 2713 40  0000 C CNN
 F 2 "Connector_PinHeader_2.54mm:PinHeader_1x08_P2.54mm_Vertical" H 7650 3550 60  0001 C CNN
@@
 $EndComp
 $Comp
-L DMPro17-rescue:M08 JP4
+L DMPro17-rescue:M08 JP3
 U 1 1 5BAC647C
 P 7650 4450
-F 0 "JP4" H 7469 3529 50  0000 C CNN
+F 0 "JP3" H 7469 3529 50  0000 C CNN
 F 1 "M08" H 7469 3613 40  0000 C CNN
 F 2 "Connector_PinHeader_2.54mm:PinHeader_1x08_P2.54mm_Vertical" H 7650 4450 60  0001 C CNN
@@
 	8050 4450 7950 4450
 $Comp
-L DMPro17-rescue:M10 JP5
+L DMPro17-rescue:M10 JP4
 U 1 1 5BAE89E7
 P 7650 5550
-F 0 "JP5" H 7469 4429 50  0000 C CNN
+F 0 "JP4" H 7469 4429 50  0000 C CNN
 F 1 "M10" H 7469 4513 40  0000 C CNN
 F 2 "Connector_PinHeader_2.54mm:PinHeader_1x10_P2.54mm_Vertical" H 7650 5550 60  0001 C CNN
@@
 Connection ~ 7950 5550
 $Comp
-L DMPro17-rescue:M06 JP6
+L DMPro17-rescue:M06 JP5
 U 1 1 5BB0CADE
 P 10600 1950
-F 0 "JP6" H 10578 1728 50  0000 L CNN
+F 0 "JP5" H 10578 1728 50  0000 L CNN
 F 1 "M06" H 10578 1644 40  0000 L CNN
 F 2 "Connector_PinHeader_2.54mm:PinHeader_1x06_P2.54mm_Vertical" H 10600 1950 60  0001 C CNN
@@
 	10150 2450 10300 2450
 $Comp
-L DMPro17-rescue:M04 JP7
+L DMPro17-rescue:M04 JP6
 U 1 1 5BB1CAA8
 P 10600 2650
-F 0 "JP7" H 10578 2528 50  0000 L CNN
+F 0 "JP6" H 10578 2528 50  0000 L CNN
 F 1 "M04" H 10578 2444 40  0000 L CNN
 F 2 "Connector_PinHeader_2.54mm:PinHeader_1x04_P2.54mm_Vertical" H 10600 2650 60  0001 C CNN
@@
 	10150 2950 10300 2950
 $Comp
-L DMPro17-rescue:M06 JP8
+L DMPro17-rescue:M06 JP7
 U 1 1 5BB28935
 P 10600 3150
-F 0 "JP8" H 10578 2928 50  0000 L CNN
+F 0 "JP7" H 10578 2928 50  0000 L CNN
 F 1 "M06" H 10578 2844 40  0000 L CNN
 F 2 "Connector_PinHeader_2.54mm:PinHeader_1x06_P2.54mm_Vertical" H 10600 3150 60  0001 C CNN
@@
 	10150 3650 10300 3650
 $Comp
-L DMPro17-rescue:M08 JP9
+L DMPro17-rescue:M08 JP8
 U 1 1 5BB3FDEB
 P 10600 3850
-F 0 "JP9" H 10578 3528 50  0000 L CNN
+F 0 "JP8" H 10578 3528 50  0000 L CNN
 F 1 "M08" H 10578 3444 40  0000 L CNN
 F 2 "Connector_PinHeader_2.54mm:PinHeader_1x08_P2.54mm_Vertical" H 10600 3850 60  0001 C CNN
@@
 F0 "PYNQ-DEBUG" 50
 F1 "PYNQ-DEBUG.sch" 50
-F2 "LED_1" I R 7400 3950 50
-F3 "LED_2" I R 7400 4050 50
-F4 "SW_1" I R 7400 4150 50
-F5 "SW_2" I R 7400 4250 50
+F2 "LED_1" I R 7400 4150 50
+F3 "LED_2" I R 7400 4250 50
+F4 "SW_1" I R 7400 3950 50
+F5 "SW_2" I R 7400 4050 50
 $EndSheet
 Connection ~ 7950 3950
@@
 Wire Wire Line
 	7400 4250 7950 4250
-Wire Wire Line
-	7650 2400 7650 2350
-Wire Wire Line
-	7650 2350 7950 2350
-Connection ~ 7950 2350
-Wire Wire Line
-	7650 2500 7650 2450
-Wire Wire Line
-	7650 2450 7950 2450
-Connection ~ 7950 2450
-Wire Wire Line
-	7650 2600 7650 2550
-Wire Wire Line
-	7650 2550 7950 2550
-Connection ~ 7950 2550
-Wire Wire Line
-	7650 2700 7650 2650
-Wire Wire Line
-	7650 2650 7950 2650
-Connection ~ 7950 2650
 $Comp
 L efm32-symbols:EFM32GG980 U1
@@
 	1    0    0    -1
 $EndComp
-Text Label 1650 3600 0    50   ~ 0
-PF10
-Text Label 1650 3500 0    50   ~ 0
-PF11
+Text Label 1650 2200 0    50   ~ 0
+PF10_ATX
+Text Label 1650 2100 0    50   ~ 0
+PF11_ARX
+Wire Wire Line
+	2600 6100 3050 6100
+Wire Wire Line
+	2600 6200 3050 6200
+Wire Wire Line
+	2600 6300 3050 6300
+Wire Wire Line
+	2600 6400 3050 6400
+Text Label 1950 4600 0    50   ~ 0
+PB11_IMU_SDA
+Text Label 1950 4700 0    50   ~ 0
+PB12_IMU_SCL
+Wire Wire Line
+	5850 3200 5250 3200
+Wire Wire Line
+	5250 3100 5850 3100
+Wire Wire Line
+	5850 3000 5250 3000
+NoConn ~ 10300 4550
+Text Label 1650 2900 0    50   ~ 0
+PB8_CRX
+Text Label 1650 3000 0    50   ~ 0
+PB7_CTX
+Text Label 1650 2600 0    50   ~ 0
+PC2_BTX
+Text Label 1650 2500 0    50   ~ 0
+PC3_BRX
+Text Label 5250 4100 0    50   ~ 0
+PF11_ARX
 Text Label 5250 4200 0    50   ~ 0
-PF10
-Text Label 5250 4100 0    50   ~ 0
-PF11
-Text Label 1650 4000 0    50   ~ 0
-PB9
-Text Label 1650 3900 0    50   ~ 0
-PB10
-Text Label 1650 4400 0    50   ~ 0
-PA3
-Text Label 1650 4300 0    50   ~ 0
-PA4
-Text Label 3050 5200 2    50   ~ 0
-PB9
+PF10_ATX
+Text Label 3050 3600 2    50   ~ 0
+PC3_BRX
+Text Label 3050 3500 2    50   ~ 0
+PC2_BTX
+Text Label 3050 4000 2    50   ~ 0
+PB8_CRX
+Text Label 3050 3900 2    50   ~ 0
+PB7_CTX
+Text Label 3050 5400 2    50   ~ 0
+PB11_IMU_SDA
+Text Label 3050 5500 2    50   ~ 0
+PB12_IMU_SCL
+Text Label 1950 4800 0    50   ~ 0
+PB10_IMU_RST
 Text Label 3050 5300 2    50   ~ 0
-PB10
-Text Label 3050 2000 2    50   ~ 0
-PA4
-Text Label 3050 1900 2    50   ~ 0
-PA3
-Wire Wire Line
-	2600 6100 3050 6100
-Wire Wire Line
-	2600 6200 3050 6200
-Wire Wire Line
-	2600 6300 3050 6300
-Wire Wire Line
-	2600 6400 3050 6400
-Wire Wire Line
-	2900 3700 3050 3700
-Wire Wire Line
-	2900 3800 3050 3800
-Wire Wire Line
-	2900 3900 3050 3900
-Text Label 1650 3300 0    50   ~ 0
-PD5
-Text Label 1650 3400 0    50   ~ 0
-PD6
-Text Label 1650 3700 0    50   ~ 0
-PB11
-Text Label 1650 3800 0    50   ~ 0
-PB12
-Text Label 1650 4100 0    50   ~ 0
-PB4
-Text Label 1650 4200 0    50   ~ 0
-PB5
-Text Label 5250 6500 0    50   ~ 0
-PD5
+PB10_IMU_RST
+Wire Wire Line
+	5250 4500 5350 4500
+Wire Wire Line
+	5250 4600 5350 4600
+Wire Wire Line
+	5250 4700 5350 4700
+Wire Wire Line
+	5250 4800 5350 4800
+Text Label 1950 4900 0    50   ~ 0
+PA9_IMU_INT
+Text Label 3050 4300 2    50   ~ 0
+PA9_IMU_INT
+Text Label 1650 2000 0    50   ~ 0
+PD7_A2
+Text Label 1650 1900 0    50   ~ 0
+PD6_A1
 Text Label 5250 6400 0    50   ~ 0
-PD6
-Text Label 3050 5400 2    50   ~ 0
-PB11
-Text Label 3050 5500 2    50   ~ 0
-PB12
-Text Label 3050 2800 2    50   ~ 0
-PB4
-Text Label 3050 2900 2    50   ~ 0
-PB5
-Wire Wire Line
-	5850 3200 5250 3200
-Wire Wire Line
-	5250 3100 5850 3100
-Wire Wire Line
-	5850 3000 5250 3000
-Wire Wire Line
-	5650 5000 5250 5000
-Wire Wire Line
-	5650 4900 5250 4900
-Text Label 5650 4700 2    50   ~ 0
-PC0
-Text Label 5650 4800 2    50   ~ 0
-PC1
+PD6_A1
+Text Label 5250 6300 0    50   ~ 0
+PD7_A2
+Text Label 1650 2700 0    50   ~ 0
+PA7_C1
+Text Label 1650 2800 0    50   ~ 0
+PA8_C2
+Text Label 3050 4100 2    50   ~ 0
+PA7_C1
+Text Label 3050 4200 2    50   ~ 0
+PA8_C2
+Text Label 1650 2400 0    50   ~ 0
+PC1_B2
+Text Label 1650 2300 0    50   ~ 0
+PC0_B1
 Text Label 3050 3300 2    50   ~ 0
-PC0
+PC0_B1
 Text Label 3050 3400 2    50   ~ 0
-PC1
+PC1_B2
 $EndSCHEMATC
