File: pcb/CLOCK.sch (KiCad schematic (older format))
At the start: 1 part, among them Y1 Crystal_GND23

Commit message: Finishe schematic, add netlist and start editing pcb design
Parts:
- Y1: footprint (none) -> Crystal:Crystal_SMD_3225-4Pin_3.2x2.5mm_HandSoldering
Changed lines of the file:
@@
 F 0 "Y1" H 6000 4050 50  0000 L CNN
 F 1 "Crystal_GND23" H 6000 3850 50  0000 L CNN
-F 2 "" H 5800 3950 50  0001 C CNN
+F 2 "Crystal:Crystal_SMD_3225-4Pin_3.2x2.5mm_HandSoldering" H 5800 3950 50  0001 C CNN
 F 3 "~" H 5800 3950 50  0001 C CNN
 	1    5800 3950
