File: pcb/DECOUPLING.sch (KiCad schematic (older format))
At the start: 12 parts

Commit message: Finishe schematic, add netlist and start editing pcb design
Parts:
- C1, C10, C2, C3, C4, C5, C6, C7, C8, C9: footprint (none) -> Capacitor_SMD:C_0603_1608Metric_Pad1.05x0.95mm_HandSolder
- L1: footprint (none) -> Inductor_SMD:L_0603_1608Metric_Pad1.05x0.95mm_HandSolder
- R5: footprint (none) -> Resistor_SMD:R_0603_1608Metric_Pad1.05x0.95mm_HandSolder
Changed lines of the file:
@@
 F 0 "C1" H 5465 5446 50  0000 L CNN
 F 1 "100n" H 5465 5355 50  0000 L CNN
-F 2 "" H 5388 5250 50  0001 C CNN
+F 2 "Capacitor_SMD:C_0603_1608Metric_Pad1.05x0.95mm_HandSolder" H 5388 5250 50  0001 C CNN
 F 3 "~" H 5350 5400 50  0001 C CNN
 	1    5350 5400
@@
 F 0 "C3" H 5815 5446 50  0000 L CNN
 F 1 "100n" H 5815 5355 50  0000 L CNN
-F 2 "" H 5738 5250 50  0001 C CNN
+F 2 "Capacitor_SMD:C_0603_1608Metric_Pad1.05x0.95mm_HandSolder" H 5738 5250 50  0001 C CNN
 F 3 "~" H 5700 5400 50  0001 C CNN
 	1    5700 5400
@@
 F 0 "C4" H 6165 5446 50  0000 L CNN
 F 1 "100n" H 6165 5355 50  0000 L CNN
-F 2 "" H 6088 5250 50  0001 C CNN
+F 2 "Capacitor_SMD:C_0603_1608Metric_Pad1.05x0.95mm_HandSolder" H 6088 5250 50  0001 C CNN
 F 3 "~" H 6050 5400 50  0001 C CNN
 	1    6050 5400
@@
 F 0 "C6" H 6515 5446 50  0000 L CNN
 F 1 "100n" H 6515 5355 50  0000 L CNN
-F 2 "" H 6438 5250 50  0001 C CNN
+F 2 "Capacitor_SMD:C_0603_1608Metric_Pad1.05x0.95mm_HandSolder" H 6438 5250 50  0001 C CNN
 F 3 "~" H 6400 5400 50  0001 C CNN
 	1    6400 5400
@@
 F 0 "C8" H 6865 5446 50  0000 L CNN
 F 1 "100n" H 6865 5355 50  0000 L CNN
-F 2 "" H 6788 5250 50  0001 C CNN
+F 2 "Capacitor_SMD:C_0603_1608Metric_Pad1.05x0.95mm_HandSolder" H 6788 5250 50  0001 C CNN
 F 3 "~" H 6750 5400 50  0001 C CNN
 	1    6750 5400
@@
 F 0 "C9" H 7215 5446 50  0000 L CNN
 F 1 "10u" H 7215 5355 50  0000 L CNN
-F 2 "" H 7138 5250 50  0001 C CNN
+F 2 "Capacitor_SMD:C_0603_1608Metric_Pad1.05x0.95mm_HandSolder" H 7138 5250 50  0001 C CNN
 F 3 "~" H 7100 5400 50  0001 C CNN
 	1    7100 5400
@@
 F 0 "C7" H 6615 3846 50  0000 L CNN
 F 1 "1uF" H 6615 3755 50  0000 L CNN
-F 2 "" H 6538 3650 50  0001 C CNN
+F 2 "Capacitor_SMD:C_0603_1608Metric_Pad1.05x0.95mm_HandSolder" H 6538 3650 50  0001 C CNN
 F 3 "~" H 6500 3800 50  0001 C CNN
 	1    6500 3800
@@
 F 0 "C5" H 6215 3846 50  0000 L CNN
 F 1 "10nF" H 6215 3755 50  0000 L CNN
-F 2 "" H 6138 3650 50  0001 C CNN
+F 2 "Capacitor_SMD:C_0603_1608Metric_Pad1.05x0.95mm_HandSolder" H 6138 3650 50  0001 C CNN
 F 3 "~" H 6100 3800 50  0001 C CNN
 	1    6100 3800
@@
 F 0 "C2" H 5815 3846 50  0000 L CNN
 F 1 "10nF" H 5815 3755 50  0000 L CNN
-F 2 "" H 5738 3650 50  0001 C CNN
+F 2 "Capacitor_SMD:C_0603_1608Metric_Pad1.05x0.95mm_HandSolder" H 5738 3650 50  0001 C CNN
 F 3 "~" H 5700 3800 50  0001 C CNN
 	1    5700 3800
@@
 F 0 "L1" H 6153 3096 50  0000 L CNN
 F 1 "742792662 " H 6153 3005 50  0000 L CNN
-F 2 "" H 6100 3050 50  0001 C CNN
+F 2 "Inductor_SMD:L_0603_1608Metric_Pad1.05x0.95mm_HandSolder" H 6100 3050 50  0001 C CNN
 F 3 "~" H 6100 3050 50  0001 C CNN
 	1    6100 3050
@@
 F 0 "R5" H 6170 3446 50  0000 L CNN
 F 1 "1" H 6170 3355 50  0000 L CNN
-F 2 "" V 6030 3400 50  0001 C CNN
+F 2 "Resistor_SMD:R_0603_1608Metric_Pad1.05x0.95mm_HandSolder" V 6030 3400 50  0001 C CNN
 F 3 "~" H 6100 3400 50  0001 C CNN
 	1    6100 3400
@@
 F 0 "C10" V 7748 4300 50  0000 C CNN
 F 1 "1uF" V 7839 4300 50  0000 C CNN
-F 2 "" H 8038 4150 50  0001 C CNN
+F 2 "Capacitor_SMD:C_0603_1608Metric_Pad1.05x0.95mm_HandSolder" H 8038 4150 50  0001 C CNN
 F 3 "~" H 8000 4300 50  0001 C CNN
 	1    8000 4300

Commit message: continue on pcb
Parts:
- C1, C10, C2, C3, C4, C5, C6, C7, C8, C9: footprint Capacitor_SMD:C_0603_1608Metric_Pad1.05x0.95mm_HandSolder -> Capacitor_SMD:C_1206_3216Metric_Pad1.42x1.75mm_HandSolder
- L1: footprint Inductor_SMD:L_0603_1608Metric_Pad1.05x0.95mm_HandSolder -> Inductor_SMD:L_1206_3216Metric_Pad1.42x1.75mm_HandSolder
- R5: footprint Resistor_SMD:R_0603_1608Metric_Pad1.05x0.95mm_HandSolder -> Resistor_SMD:R_1206_3216Metric_Pad1.42x1.75mm_HandSolder
Changed lines of the file:
@@
 F 0 "C1" H 5465 5446 50  0000 L CNN
 F 1 "100n" H 5465 5355 50  0000 L CNN
-F 2 "Capacitor_SMD:C_0603_1608Metric_Pad1.05x0.95mm_HandSolder" H 5388 5250 50  0001 C CNN
+F 2 "Capacitor_SMD:C_1206_3216Metric_Pad1.42x1.75mm_HandSolder" H 5388 5250 50  0001 C CNN
 F 3 "~" H 5350 5400 50  0001 C CNN
 	1    5350 5400
@@
 F 0 "C3" H 5815 5446 50  0000 L CNN
 F 1 "100n" H 5815 5355 50  0000 L CNN
-F 2 "Capacitor_SMD:C_0603_1608Metric_Pad1.05x0.95mm_HandSolder" H 5738 5250 50  0001 C CNN
+F 2 "Capacitor_SMD:C_1206_3216Metric_Pad1.42x1.75mm_HandSolder" H 5738 5250 50  0001 C CNN
 F 3 "~" H 5700 5400 50  0001 C CNN
 	1    5700 5400
@@
 F 0 "C4" H 6165 5446 50  0000 L CNN
 F 1 "100n" H 6165 5355 50  0000 L CNN
-F 2 "Capacitor_SMD:C_0603_1608Metric_Pad1.05x0.95mm_HandSolder" H 6088 5250 50  0001 C CNN
+F 2 "Capacitor_SMD:C_1206_3216Metric_Pad1.42x1.75mm_HandSolder" H 6088 5250 50  0001 C CNN
 F 3 "~" H 6050 5400 50  0001 C CNN
 	1    6050 5400
@@
 F 0 "C6" H 6515 5446 50  0000 L CNN
 F 1 "100n" H 6515 5355 50  0000 L CNN
-F 2 "Capacitor_SMD:C_0603_1608Metric_Pad1.05x0.95mm_HandSolder" H 6438 5250 50  0001 C CNN
+F 2 "Capacitor_SMD:C_1206_3216Metric_Pad1.42x1.75mm_HandSolder" H 6438 5250 50  0001 C CNN
 F 3 "~" H 6400 5400 50  0001 C CNN
 	1    6400 5400
@@
 F 0 "C8" H 6865 5446 50  0000 L CNN
 F 1 "100n" H 6865 5355 50  0000 L CNN
-F 2 "Capacitor_SMD:C_0603_1608Metric_Pad1.05x0.95mm_HandSolder" H 6788 5250 50  0001 C CNN
+F 2 "Capacitor_SMD:C_1206_3216Metric_Pad1.42x1.75mm_HandSolder" H 6788 5250 50  0001 C CNN
 F 3 "~" H 6750 5400 50  0001 C CNN
 	1    6750 5400
@@
 F 0 "C9" H 7215 5446 50  0000 L CNN
 F 1 "10u" H 7215 5355 50  0000 L CNN
-F 2 "Capacitor_SMD:C_0603_1608Metric_Pad1.05x0.95mm_HandSolder" H 7138 5250 50  0001 C CNN
+F 2 "Capacitor_SMD:C_1206_3216Metric_Pad1.42x1.75mm_HandSolder" H 7138 5250 50  0001 C CNN
 F 3 "~" H 7100 5400 50  0001 C CNN
 	1    7100 5400
@@
 F 0 "C7" H 6615 3846 50  0000 L CNN
 F 1 "1uF" H 6615 3755 50  0000 L CNN
-F 2 "Capacitor_SMD:C_0603_1608Metric_Pad1.05x0.95mm_HandSolder" H 6538 3650 50  0001 C CNN
+F 2 "Capacitor_SMD:C_1206_3216Metric_Pad1.42x1.75mm_HandSolder" H 6538 3650 50  0001 C CNN
 F 3 "~" H 6500 3800 50  0001 C CNN
 	1    6500 3800
@@
 F 0 "C5" H 6215 3846 50  0000 L CNN
 F 1 "10nF" H 6215 3755 50  0000 L CNN
-F 2 "Capacitor_SMD:C_0603_1608Metric_Pad1.05x0.95mm_HandSolder" H 6138 3650 50  0001 C CNN
+F 2 "Capacitor_SMD:C_1206_3216Metric_Pad1.42x1.75mm_HandSolder" H 6138 3650 50  0001 C CNN
 F 3 "~" H 6100 3800 50  0001 C CNN
 	1    6100 3800
@@
 F 0 "C2" H 5815 3846 50  0000 L CNN
 F 1 "10nF" H 5815 3755 50  0000 L CNN
-F 2 "Capacitor_SMD:C_0603_1608Metric_Pad1.05x0.95mm_HandSolder" H 5738 3650 50  0001 C CNN
+F 2 "Capacitor_SMD:C_1206_3216Metric_Pad1.42x1.75mm_HandSolder" H 5738 3650 50  0001 C CNN
 F 3 "~" H 5700 3800 50  0001 C CNN
 	1    5700 3800
@@
 F 0 "L1" H 6153 3096 50  0000 L CNN
 F 1 "742792662 " H 6153 3005 50  0000 L CNN
-F 2 "Inductor_SMD:L_0603_1608Metric_Pad1.05x0.95mm_HandSolder" H 6100 3050 50  0001 C CNN
+F 2 "Inductor_SMD:L_1206_3216Metric_Pad1.42x1.75mm_HandSolder" H 6100 3050 50  0001 C CNN
 F 3 "~" H 6100 3050 50  0001 C CNN
 	1    6100 3050
@@
 F 0 "R5" H 6170 3446 50  0000 L CNN
 F 1 "1" H 6170 3355 50  0000 L CNN
-F 2 "Resistor_SMD:R_0603_1608Metric_Pad1.05x0.95mm_HandSolder" V 6030 3400 50  0001 C CNN
+F 2 "Resistor_SMD:R_1206_3216Metric_Pad1.42x1.75mm_HandSolder" V 6030 3400 50  0001 C CNN
 F 3 "~" H 6100 3400 50  0001 C CNN
 	1    6100 3400
@@
 F 0 "C10" V 7748 4300 50  0000 C CNN
 F 1 "1uF" V 7839 4300 50  0000 C CNN
-F 2 "Capacitor_SMD:C_0603_1608Metric_Pad1.05x0.95mm_HandSolder" H 8038 4150 50  0001 C CNN
+F 2 "Capacitor_SMD:C_1206_3216Metric_Pad1.42x1.75mm_HandSolder" H 8038 4150 50  0001 C CNN
 F 3 "~" H 8000 4300 50  0001 C CNN
 	1    8000 4300
