File: pcb/EFM_DEBUG.sch (KiCad schematic (older format))
At the start: 8 parts, among them SW1 SW_PUSHBUTTON, SW2 SW_PUSHBUTTON

Commit message: Finishe schematic, add netlist and start editing pcb design
Parts:
- D1, D2: footprint (none) -> LED_SMD:LED_0603_1608Metric_Pad1.05x0.95mm_HandSolder
- R1, R2, R3, R4: footprint (none) -> Resistor_SMD:R_0603_1608Metric_Pad1.05x0.95mm_HandSolder
- SW1, SW2: footprint (none) -> myfootprint:SW_PUSHBUTTON_SMD
Changed lines of the file:
@@
 F 0 "D1" V 6238 3083 50  0000 R CNN
 F 1 "LED" V 6147 3083 50  0000 R CNN
-F 2 "" H 6200 3200 50  0001 C CNN
+F 2 "LED_SMD:LED_0603_1608Metric_Pad1.05x0.95mm_HandSolder" H 6200 3200 50  0001 C CNN
 F 3 "~" H 6200 3200 50  0001 C CNN
 	1    6200 3200
@@
 F 0 "D2" V 6638 3083 50  0000 R CNN
 F 1 "LED" V 6547 3083 50  0000 R CNN
-F 2 "" H 6600 3200 50  0001 C CNN
+F 2 "LED_SMD:LED_0603_1608Metric_Pad1.05x0.95mm_HandSolder" H 6600 3200 50  0001 C CNN
 F 3 "~" H 6600 3200 50  0001 C CNN
 	1    6600 3200
@@
 F 0 "R3" H 6270 2796 50  0000 L CNN
 F 1 "R" H 6270 2705 50  0000 L CNN
-F 2 "" V 6130 2750 50  0001 C CNN
+F 2 "Resistor_SMD:R_0603_1608Metric_Pad1.05x0.95mm_HandSolder" V 6130 2750 50  0001 C CNN
 F 3 "~" H 6200 2750 50  0001 C CNN
 	1    6200 2750
@@
 F 0 "R4" H 6670 2796 50  0000 L CNN
 F 1 "R" H 6670 2705 50  0000 L CNN
-F 2 "" V 6530 2750 50  0001 C CNN
+F 2 "Resistor_SMD:R_0603_1608Metric_Pad1.05x0.95mm_HandSolder" V 6530 2750 50  0001 C CNN
 F 3 "~" H 6600 2750 50  0001 C CNN
 	1    6600 2750
@@
 F 0 "SW1" H 4100 3165 50  0000 C CNN
 F 1 "SW_PUSHBUTTON" H 4100 3074 50  0000 C CNN
-F 2 "" H 4100 2900 60  0001 C CNN
+F 2 "myfootprint:SW_PUSHBUTTON_SMD" H 4100 2900 60  0001 C CNN
 F 3 "" H 4100 2900 60  0000 C CNN
 	1    4100 2900
@@
 F 0 "R1" H 3620 2646 50  0000 L CNN
 F 1 "R" H 3620 2555 50  0000 L CNN
-F 2 "" V 3480 2600 50  0001 C CNN
+F 2 "Resistor_SMD:R_0603_1608Metric_Pad1.05x0.95mm_HandSolder" V 3480 2600 50  0001 C CNN
 F 3 "~" H 3550 2600 50  0001 C CNN
 	1    3550 2600
@@
 F 0 "SW2" H 4100 4115 50  0000 C CNN
 F 1 "SW_PUSHBUTTON" H 4100 4024 50  0000 C CNN
-F 2 "" H 4100 3850 60  0001 C CNN
+F 2 "myfootprint:SW_PUSHBUTTON_SMD" H 4100 3850 60  0001 C CNN
 F 3 "" H 4100 3850 60  0000 C CNN
 	1    4100 3850
@@
 F 0 "R2" H 3620 3596 50  0000 L CNN
 F 1 "R" H 3620 3505 50  0000 L CNN
-F 2 "" V 3480 3550 50  0001 C CNN
+F 2 "Resistor_SMD:R_0603_1608Metric_Pad1.05x0.95mm_HandSolder" V 3480 3550 50  0001 C CNN
 F 3 "~" H 3550 3550 50  0001 C CNN
 	1    3550 3550

Commit message: continue on pcb
Parts:
- D1, D2: footprint LED_SMD:LED_0603_1608Metric_Pad1.05x0.95mm_HandSolder -> LED_SMD:LED_1206_3216Metric_Pad1.42x1.75mm_HandSolder
- R1, R2, R3, R4: footprint Resistor_SMD:R_0603_1608Metric_Pad1.05x0.95mm_HandSolder -> Resistor_SMD:R_1206_3216Metric_Pad1.42x1.75mm_HandSolder
Changed lines of the file:
@@
 F 0 "D1" V 6238 3083 50  0000 R CNN
 F 1 "LED" V 6147 3083 50  0000 R CNN
-F 2 "LED_SMD:LED_0603_1608Metric_Pad1.05x0.95mm_HandSolder" H 6200 3200 50  0001 C CNN
+F 2 "LED_SMD:LED_1206_3216Metric_Pad1.42x1.75mm_HandSolder" H 6200 3200 50  0001 C CNN
 F 3 "~" H 6200 3200 50  0001 C CNN
 	1    6200 3200
@@
 F 0 "D2" V 6638 3083 50  0000 R CNN
 F 1 "LED" V 6547 3083 50  0000 R CNN
-F 2 "LED_SMD:LED_0603_1608Metric_Pad1.05x0.95mm_HandSolder" H 6600 3200 50  0001 C CNN
+F 2 "LED_SMD:LED_1206_3216Metric_Pad1.42x1.75mm_HandSolder" H 6600 3200 50  0001 C CNN
 F 3 "~" H 6600 3200 50  0001 C CNN
 	1    6600 3200
@@
 F 0 "R3" H 6270 2796 50  0000 L CNN
 F 1 "R" H 6270 2705 50  0000 L CNN
-F 2 "Resistor_SMD:R_0603_1608Metric_Pad1.05x0.95mm_HandSolder" V 6130 2750 50  0001 C CNN
+F 2 "Resistor_SMD:R_1206_3216Metric_Pad1.42x1.75mm_HandSolder" V 6130 2750 50  0001 C CNN
 F 3 "~" H 6200 2750 50  0001 C CNN
 	1    6200 2750
@@
 F 0 "R4" H 6670 2796 50  0000 L CNN
 F 1 "R" H 6670 2705 50  0000 L CNN
-F 2 "Resistor_SMD:R_0603_1608Metric_Pad1.05x0.95mm_HandSolder" V 6530 2750 50  0001 C CNN
+F 2 "Resistor_SMD:R_1206_3216Metric_Pad1.42x1.75mm_HandSolder" V 6530 2750 50  0001 C CNN
 F 3 "~" H 6600 2750 50  0001 C CNN
 	1    6600 2750
@@
 F 0 "R1" H 3620 2646 50  0000 L CNN
 F 1 "R" H 3620 2555 50  0000 L CNN
-F 2 "Resistor_SMD:R_0603_1608Metric_Pad1.05x0.95mm_HandSolder" V 3480 2600 50  0001 C CNN
+F 2 "Resistor_SMD:R_1206_3216Metric_Pad1.42x1.75mm_HandSolder" V 3480 2600 50  0001 C CNN
 F 3 "~" H 3550 2600 50  0001 C CNN
 	1    3550 2600
@@
 F 0 "R2" H 3620 3596 50  0000 L CNN
 F 1 "R" H 3620 3505 50  0000 L CNN
-F 2 "Resistor_SMD:R_0603_1608Metric_Pad1.05x0.95mm_HandSolder" V 3480 3550 50  0001 C CNN
+F 2 "Resistor_SMD:R_1206_3216Metric_Pad1.42x1.75mm_HandSolder" V 3480 3550 50  0001 C CNN
 F 3 "~" H 3550 3550 50  0001 C CNN
 	1    3550 3550
