File: pcb/PYNQ-DEBUG.sch (KiCad schematic (older format))
At the start: 8 parts

Commit message: Finishe schematic, add netlist and start editing pcb design
Parts:
- D3, D4: renamed from D?; footprint (none) -> LED_SMD:LED_0603_1608Metric_Pad1.05x0.95mm_HandSolder
- R14, R15, R16, R17: renamed from R?; footprint (none) -> Resistor_SMD:R_0603_1608Metric_Pad1.05x0.95mm_HandSolder
- SW3, SW4: renamed from SW?; footprint (none) -> myfootprint:SW_PUSHBUTTON_SMD
Changed lines of the file:
@@
 AR Path="/5BA41DB8/5BB6E88B" Ref="D?"  Part="1"
 AR Path="/5BB20D15/5BB6E88B" Ref="D?"  Part="1"
-AR Path="/5BB6E330/5BB6E88B" Ref="D?"  Part="1"
-F 0 "D?" V 6888 3783 50  0000 R CNN
+AR Path="/5BB6E330/5BB6E88B" Ref="D3"  Part="1"
+F 0 "D3" V 6888 3783 50  0000 R CNN
 F 1 "LED" V 6797 3783 50  0000 R CNN
-F 2 "" H 6850 3900 50  0001 C CNN
+F 2 "LED_SMD:LED_0603_1608Metric_Pad1.05x0.95mm_HandSolder" H 6850 3900 50  0001 C CNN
 F 3 "~" H 6850 3900 50  0001 C CNN
 	1    6850 3900
@@
 AR Path="/5BA41DB8/5BB6E892" Ref="D?"  Part="1"
 AR Path="/5BB20D15/5BB6E892" Ref="D?"  Part="1"
-AR Path="/5BB6E330/5BB6E892" Ref="D?"  Part="1"
-F 0 "D?" V 7288 3783 50  0000 R CNN
+AR Path="/5BB6E330/5BB6E892" Ref="D4"  Part="1"
+F 0 "D4" V 7288 3783 50  0000 R CNN
 F 1 "LED" V 7197 3783 50  0000 R CNN
-F 2 "" H 7250 3900 50  0001 C CNN
+F 2 "LED_SMD:LED_0603_1608Metric_Pad1.05x0.95mm_HandSolder" H 7250 3900 50  0001 C CNN
 F 3 "~" H 7250 3900 50  0001 C CNN
 	1    7250 3900
@@
 AR Path="/5BA41DB8/5BB6E899" Ref="R?"  Part="1"
 AR Path="/5BB20D15/5BB6E899" Ref="R?"  Part="1"
-AR Path="/5BB6E330/5BB6E899" Ref="R?"  Part="1"
-F 0 "R?" H 6920 3496 50  0000 L CNN
+AR Path="/5BB6E330/5BB6E899" Ref="R16"  Part="1"
+F 0 "R16" H 6920 3496 50  0000 L CNN
 F 1 "R" H 6920 3405 50  0000 L CNN
-F 2 "" V 6780 3450 50  0001 C CNN
+F 2 "Resistor_SMD:R_0603_1608Metric_Pad1.05x0.95mm_HandSolder" V 6780 3450 50  0001 C CNN
 F 3 "~" H 6850 3450 50  0001 C CNN
 	1    6850 3450
@@
 AR Path="/5BA41DB8/5BB6E8A0" Ref="R?"  Part="1"
 AR Path="/5BB20D15/5BB6E8A0" Ref="R?"  Part="1"
-AR Path="/5BB6E330/5BB6E8A0" Ref="R?"  Part="1"
-F 0 "R?" H 7320 3496 50  0000 L CNN
+AR Path="/5BB6E330/5BB6E8A0" Ref="R17"  Part="1"
+F 0 "R17" H 7320 3496 50  0000 L CNN
 F 1 "R" H 7320 3405 50  0000 L CNN
-F 2 "" V 7180 3450 50  0001 C CNN
+F 2 "Resistor_SMD:R_0603_1608Metric_Pad1.05x0.95mm_HandSolder" V 7180 3450 50  0001 C CNN
 F 3 "~" H 7250 3450 50  0001 C CNN
 	1    7250 3450
@@
 AR Path="/5BA41DB8/5BB6E8AD" Ref="#PWR?"  Part="1"
 AR Path="/5BB20D15/5BB6E8AD" Ref="#PWR?"  Part="1"
-AR Path="/5BB6E330/5BB6E8AD" Ref="#PWR?"  Part="1"
-F 0 "#PWR?" H 6850 3950 50  0001 C CNN
+AR Path="/5BB6E330/5BB6E8AD" Ref="#PWR043"  Part="1"
+F 0 "#PWR043" H 6850 3950 50  0001 C CNN
 F 1 "GND" H 6855 4027 50  0000 C CNN
 F 2 "" H 6850 4200 50  0001 C CNN
@@
 AR Path="/5BA41DB8/5BB6E8B3" Ref="#PWR?"  Part="1"
 AR Path="/5BB20D15/5BB6E8B3" Ref="#PWR?"  Part="1"
-AR Path="/5BB6E330/5BB6E8B3" Ref="#PWR?"  Part="1"
-F 0 "#PWR?" H 7250 3950 50  0001 C CNN
+AR Path="/5BB6E330/5BB6E8B3" Ref="#PWR044"  Part="1"
+F 0 "#PWR044" H 7250 3950 50  0001 C CNN
 F 1 "GND" H 7255 4027 50  0000 C CNN
 F 2 "" H 7250 4200 50  0001 C CNN
@@
 AR Path="/5BA41DB8/5BB6E8BB" Ref="SW?"  Part="1"
 AR Path="/5BB20D15/5BB6E8BB" Ref="SW?"  Part="1"
-AR Path="/5BB6E330/5BB6E8BB" Ref="SW?"  Part="1"
-F 0 "SW?" H 4750 3865 50  0000 C CNN
+AR Path="/5BB6E330/5BB6E8BB" Ref="SW3"  Part="1"
+F 0 "SW3" H 4750 3865 50  0000 C CNN
 F 1 "SW_PUSHBUTTON" H 4750 3774 50  0000 C CNN
-F 2 "" H 4750 3600 60  0001 C CNN
+F 2 "myfootprint:SW_PUSHBUTTON_SMD" H 4750 3600 60  0001 C CNN
 F 3 "" H 4750 3600 60  0000 C CNN
 	1    4750 3600
@@
 AR Path="/5BA41DB8/5BB6E8C2" Ref="R?"  Part="1"
 AR Path="/5BB20D15/5BB6E8C2" Ref="R?"  Part="1"
-AR Path="/5BB6E330/5BB6E8C2" Ref="R?"  Part="1"
-F 0 "R?" H 4270 3346 50  0000 L CNN
+AR Path="/5BB6E330/5BB6E8C2" Ref="R14"  Part="1"
+F 0 "R14" H 4270 3346 50  0000 L CNN
 F 1 "R" H 4270 3255 50  0000 L CNN
-F 2 "" V 4130 3300 50  0001 C CNN
+F 2 "Resistor_SMD:R_0603_1608Metric_Pad1.05x0.95mm_HandSolder" V 4130 3300 50  0001 C CNN
 F 3 "~" H 4200 3300 50  0001 C CNN
 	1    4200 3300
@@
 AR Path="/5BA41DB8/5BB6E8C9" Ref="#PWR?"  Part="1"
 AR Path="/5BB20D15/5BB6E8C9" Ref="#PWR?"  Part="1"
-AR Path="/5BB6E330/5BB6E8C9" Ref="#PWR?"  Part="1"
-F 0 "#PWR?" H 5250 3350 50  0001 C CNN
+AR Path="/5BB6E330/5BB6E8C9" Ref="#PWR041"  Part="1"
+F 0 "#PWR041" H 5250 3350 50  0001 C CNN
 F 1 "GND" V 5255 3472 50  0000 R CNN
 F 2 "" H 5250 3600 50  0001 C CNN
@@
 AR Path="/5BA41DB8/5BB6E8D2" Ref="#PWR?"  Part="1"
 AR Path="/5BB20D15/5BB6E8D2" Ref="#PWR?"  Part="1"
-AR Path="/5BB6E330/5BB6E8D2" Ref="#PWR?"  Part="1"
-F 0 "#PWR?" H 4200 2850 50  0001 C CNN
+AR Path="/5BB6E330/5BB6E8D2" Ref="#PWR039"  Part="1"
+F 0 "#PWR039" H 4200 2850 50  0001 C CNN
 F 1 "+3.3V" H 4215 3173 50  0000 C CNN
 F 2 "" H 4200 3000 50  0001 C CNN
@@
 AR Path="/5BA41DB8/5BB6E8DC" Ref="SW?"  Part="1"
 AR Path="/5BB20D15/5BB6E8DC" Ref="SW?"  Part="1"
-AR Path="/5BB6E330/5BB6E8DC" Ref="SW?"  Part="1"
-F 0 "SW?" H 4750 4815 50  0000 C CNN
+AR Path="/5BB6E330/5BB6E8DC" Ref="SW4"  Part="1"
+F 0 "SW4" H 4750 4815 50  0000 C CNN
 F 1 "SW_PUSHBUTTON" H 4750 4724 50  0000 C CNN
-F 2 "" H 4750 4550 60  0001 C CNN
+F 2 "myfootprint:SW_PUSHBUTTON_SMD" H 4750 4550 60  0001 C CNN
 F 3 "" H 4750 4550 60  0000 C CNN
 	1    4750 4550
@@
 AR Path="/5BA41DB8/5BB6E8E3" Ref="R?"  Part="1"
 AR Path="/5BB20D15/5BB6E8E3" Ref="R?"  Part="1"
-AR Path="/5BB6E330/5BB6E8E3" Ref="R?"  Part="1"
-F 0 "R?" H 4270 4296 50  0000 L CNN
+AR Path="/5BB6E330/5BB6E8E3" Ref="R15"  Part="1"
+F 0 "R15" H 4270 4296 50  0000 L CNN
 F 1 "R" H 4270 4205 50  0000 L CNN
-F 2 "" V 4130 4250 50  0001 C CNN
+F 2 "Resistor_SMD:R_0603_1608Metric_Pad1.05x0.95mm_HandSolder" V 4130 4250 50  0001 C CNN
 F 3 "~" H 4200 4250 50  0001 C CNN
 	1    4200 4250
@@
 AR Path="/5BA41DB8/5BB6E8EA" Ref="#PWR?"  Part="1"
 AR Path="/5BB20D15/5BB6E8EA" Ref="#PWR?"  Part="1"
-AR Path="/5BB6E330/5BB6E8EA" Ref="#PWR?"  Part="1"
-F 0 "#PWR?" H 5250 4300 50  0001 C CNN
+AR Path="/5BB6E330/5BB6E8EA" Ref="#PWR042"  Part="1"
+F 0 "#PWR042" H 5250 4300 50  0001 C CNN
 F 1 "GND" V 5255 4422 50  0000 R CNN
 F 2 "" H 5250 4550 50  0001 C CNN
@@
 AR Path="/5BA41DB8/5BB6E8F3" Ref="#PWR?"  Part="1"
 AR Path="/5BB20D15/5BB6E8F3" Ref="#PWR?"  Part="1"
-AR Path="/5BB6E330/5BB6E8F3" Ref="#PWR?"  Part="1"
-F 0 "#PWR?" H 4200 3800 50  0001 C CNN
+AR Path="/5BB6E330/5BB6E8F3" Ref="#PWR040"  Part="1"
+F 0 "#PWR040" H 4200 3800 50  0001 C CNN
 F 1 "+3.3V" H 4215 4123 50  0000 C CNN
 F 2 "" H 4200 3950 50  0001 C CNN

Commit message: continue on pcb
Parts:
- D3, D4: footprint LED_SMD:LED_0603_1608Metric_Pad1.05x0.95mm_HandSolder -> LED_SMD:LED_1206_3216Metric_Pad1.42x1.75mm_HandSolder
- R14, R15, R16, R17: footprint Resistor_SMD:R_0603_1608Metric_Pad1.05x0.95mm_HandSolder -> Resistor_SMD:R_1206_3216Metric_Pad1.42x1.75mm_HandSolder
Changed lines of the file:
@@
 F 0 "D3" V 6888 3783 50  0000 R CNN
 F 1 "LED" V 6797 3783 50  0000 R CNN
-F 2 "LED_SMD:LED_0603_1608Metric_Pad1.05x0.95mm_HandSolder" H 6850 3900 50  0001 C CNN
+F 2 "LED_SMD:LED_1206_3216Metric_Pad1.42x1.75mm_HandSolder" H 6850 3900 50  0001 C CNN
 F 3 "~" H 6850 3900 50  0001 C CNN
 	1    6850 3900
@@
 F 0 "D4" V 7288 3783 50  0000 R CNN
 F 1 "LED" V 7197 3783 50  0000 R CNN
-F 2 "LED_SMD:LED_0603_1608Metric_Pad1.05x0.95mm_HandSolder" H 7250 3900 50  0001 C CNN
+F 2 "LED_SMD:LED_1206_3216Metric_Pad1.42x1.75mm_HandSolder" H 7250 3900 50  0001 C CNN
 F 3 "~" H 7250 3900 50  0001 C CNN
 	1    7250 3900
@@
 F 0 "R16" H 6920 3496 50  0000 L CNN
 F 1 "R" H 6920 3405 50  0000 L CNN
-F 2 "Resistor_SMD:R_0603_1608Metric_Pad1.05x0.95mm_HandSolder" V 6780 3450 50  0001 C CNN
+F 2 "Resistor_SMD:R_1206_3216Metric_Pad1.42x1.75mm_HandSolder" V 6780 3450 50  0001 C CNN
 F 3 "~" H 6850 3450 50  0001 C CNN
 	1    6850 3450
@@
 F 0 "R17" H 7320 3496 50  0000 L CNN
 F 1 "R" H 7320 3405 50  0000 L CNN
-F 2 "Resistor_SMD:R_0603_1608Metric_Pad1.05x0.95mm_HandSolder" V 7180 3450 50  0001 C CNN
+F 2 "Resistor_SMD:R_1206_3216Metric_Pad1.42x1.75mm_HandSolder" V 7180 3450 50  0001 C CNN
 F 3 "~" H 7250 3450 50  0001 C CNN
 	1    7250 3450
@@
 F 0 "R14" H 4270 3346 50  0000 L CNN
 F 1 "R" H 4270 3255 50  0000 L CNN
-F 2 "Resistor_SMD:R_0603_1608Metric_Pad1.05x0.95mm_HandSolder" V 4130 3300 50  0001 C CNN
+F 2 "Resistor_SMD:R_1206_3216Metric_Pad1.42x1.75mm_HandSolder" V 4130 3300 50  0001 C CNN
 F 3 "~" H 4200 3300 50  0001 C CNN
 	1    4200 3300
@@
 F 0 "R15" H 4270 4296 50  0000 L CNN
 F 1 "R" H 4270 4205 50  0000 L CNN
-F 2 "Resistor_SMD:R_0603_1608Metric_Pad1.05x0.95mm_HandSolder" V 4130 4250 50  0001 C CNN
+F 2 "Resistor_SMD:R_1206_3216Metric_Pad1.42x1.75mm_HandSolder" V 4130 4250 50  0001 C CNN
 F 3 "~" H 4200 4250 50  0001 C CNN
 	1    4200 4250

Commit message: Think it is somewhat finished
Parts:
- renumbered R14 to R32, R15 to R33, R16 to R34, R17 to R35, SW3 to SW12, SW4 to SW13
Changed lines of the file:
@@
 AR Path="/5BA41DB8/5BB6E899" Ref="R?"  Part="1"
 AR Path="/5BB20D15/5BB6E899" Ref="R?"  Part="1"
-AR Path="/5BB6E330/5BB6E899" Ref="R16"  Part="1"
-F 0 "R16" H 6920 3496 50  0000 L CNN
+AR Path="/5BB6E330/5BB6E899" Ref="R34"  Part="1"
+F 0 "R34" H 6920 3496 50  0000 L CNN
 F 1 "R" H 6920 3405 50  0000 L CNN
 F 2 "Resistor_SMD:R_1206_3216Metric_Pad1.42x1.75mm_HandSolder" V 6780 3450 50  0001 C CNN
@@
 AR Path="/5BA41DB8/5BB6E8A0" Ref="R?"  Part="1"
 AR Path="/5BB20D15/5BB6E8A0" Ref="R?"  Part="1"
-AR Path="/5BB6E330/5BB6E8A0" Ref="R17"  Part="1"
-F 0 "R17" H 7320 3496 50  0000 L CNN
+AR Path="/5BB6E330/5BB6E8A0" Ref="R35"  Part="1"
+F 0 "R35" H 7320 3496 50  0000 L CNN
 F 1 "R" H 7320 3405 50  0000 L CNN
 F 2 "Resistor_SMD:R_1206_3216Metric_Pad1.42x1.75mm_HandSolder" V 7180 3450 50  0001 C CNN
@@
 AR Path="/5BA41DB8/5BB6E8AD" Ref="#PWR?"  Part="1"
 AR Path="/5BB20D15/5BB6E8AD" Ref="#PWR?"  Part="1"
-AR Path="/5BB6E330/5BB6E8AD" Ref="#PWR043"  Part="1"
-F 0 "#PWR043" H 6850 3950 50  0001 C CNN
+AR Path="/5BB6E330/5BB6E8AD" Ref="#PWR075"  Part="1"
+F 0 "#PWR075" H 6850 3950 50  0001 C CNN
 F 1 "GND" H 6855 4027 50  0000 C CNN
 F 2 "" H 6850 4200 50  0001 C CNN
@@
 AR Path="/5BA41DB8/5BB6E8B3" Ref="#PWR?"  Part="1"
 AR Path="/5BB20D15/5BB6E8B3" Ref="#PWR?"  Part="1"
-AR Path="/5BB6E330/5BB6E8B3" Ref="#PWR044"  Part="1"
-F 0 "#PWR044" H 7250 3950 50  0001 C CNN
+AR Path="/5BB6E330/5BB6E8B3" Ref="#PWR076"  Part="1"
+F 0 "#PWR076" H 7250 3950 50  0001 C CNN
 F 1 "GND" H 7255 4027 50  0000 C CNN
 F 2 "" H 7250 4200 50  0001 C CNN
@@
 AR Path="/5BA41DB8/5BB6E8BB" Ref="SW?"  Part="1"
 AR Path="/5BB20D15/5BB6E8BB" Ref="SW?"  Part="1"
-AR Path="/5BB6E330/5BB6E8BB" Ref="SW3"  Part="1"
-F 0 "SW3" H 4750 3865 50  0000 C CNN
+AR Path="/5BB6E330/5BB6E8BB" Ref="SW12"  Part="1"
+F 0 "SW12" H 4750 3865 50  0000 C CNN
 F 1 "SW_PUSHBUTTON" H 4750 3774 50  0000 C CNN
 F 2 "myfootprint:SW_PUSHBUTTON_SMD" H 4750 3600 60  0001 C CNN
@@
 AR Path="/5BA41DB8/5BB6E8C2" Ref="R?"  Part="1"
 AR Path="/5BB20D15/5BB6E8C2" Ref="R?"  Part="1"
-AR Path="/5BB6E330/5BB6E8C2" Ref="R14"  Part="1"
-F 0 "R14" H 4270 3346 50  0000 L CNN
+AR Path="/5BB6E330/5BB6E8C2" Ref="R32"  Part="1"
+F 0 "R32" H 4270 3346 50  0000 L CNN
 F 1 "R" H 4270 3255 50  0000 L CNN
 F 2 "Resistor_SMD:R_1206_3216Metric_Pad1.42x1.75mm_HandSolder" V 4130 3300 50  0001 C CNN
@@
 AR Path="/5BA41DB8/5BB6E8C9" Ref="#PWR?"  Part="1"
 AR Path="/5BB20D15/5BB6E8C9" Ref="#PWR?"  Part="1"
-AR Path="/5BB6E330/5BB6E8C9" Ref="#PWR041"  Part="1"
-F 0 "#PWR041" H 5250 3350 50  0001 C CNN
+AR Path="/5BB6E330/5BB6E8C9" Ref="#PWR073"  Part="1"
+F 0 "#PWR073" H 5250 3350 50  0001 C CNN
 F 1 "GND" V 5255 3472 50  0000 R CNN
 F 2 "" H 5250 3600 50  0001 C CNN
@@
 AR Path="/5BA41DB8/5BB6E8D2" Ref="#PWR?"  Part="1"
 AR Path="/5BB20D15/5BB6E8D2" Ref="#PWR?"  Part="1"
-AR Path="/5BB6E330/5BB6E8D2" Ref="#PWR039"  Part="1"
-F 0 "#PWR039" H 4200 2850 50  0001 C CNN
+AR Path="/5BB6E330/5BB6E8D2" Ref="#PWR071"  Part="1"
+F 0 "#PWR071" H 4200 2850 50  0001 C CNN
 F 1 "+3.3V" H 4215 3173 50  0000 C CNN
 F 2 "" H 4200 3000 50  0001 C CNN
@@
 AR Path="/5BA41DB8/5BB6E8DC" Ref="SW?"  Part="1"
 AR Path="/5BB20D15/5BB6E8DC" Ref="SW?"  Part="1"
-AR Path="/5BB6E330/5BB6E8DC" Ref="SW4"  Part="1"
-F 0 "SW4" H 4750 4815 50  0000 C CNN
+AR Path="/5BB6E330/5BB6E8DC" Ref="SW13"  Part="1"
+F 0 "SW13" H 4750 4815 50  0000 C CNN
 F 1 "SW_PUSHBUTTON" H 4750 4724 50  0000 C CNN
 F 2 "myfootprint:SW_PUSHBUTTON_SMD" H 4750 4550 60  0001 C CNN
@@
 AR Path="/5BA41DB8/5BB6E8E3" Ref="R?"  Part="1"
 AR Path="/5BB20D15/5BB6E8E3" Ref="R?"  Part="1"
-AR Path="/5BB6E330/5BB6E8E3" Ref="R15"  Part="1"
-F 0 "R15" H 4270 4296 50  0000 L CNN
+AR Path="/5BB6E330/5BB6E8E3" Ref="R33"  Part="1"
+F 0 "R33" H 4270 4296 50  0000 L CNN
 F 1 "R" H 4270 4205 50  0000 L CNN
 F 2 "Resistor_SMD:R_1206_3216Metric_Pad1.42x1.75mm_HandSolder" V 4130 4250 50  0001 C CNN
@@
 AR Path="/5BA41DB8/5BB6E8EA" Ref="#PWR?"  Part="1"
 AR Path="/5BB20D15/5BB6E8EA" Ref="#PWR?"  Part="1"
-AR Path="/5BB6E330/5BB6E8EA" Ref="#PWR042"  Part="1"
-F 0 "#PWR042" H 5250 4300 50  0001 C CNN
+AR Path="/5BB6E330/5BB6E8EA" Ref="#PWR074"  Part="1"
+F 0 "#PWR074" H 5250 4300 50  0001 C CNN
 F 1 "GND" V 5255 4422 50  0000 R CNN
 F 2 "" H 5250 4550 50  0001 C CNN
@@
 AR Path="/5BA41DB8/5BB6E8F3" Ref="#PWR?"  Part="1"
 AR Path="/5BB20D15/5BB6E8F3" Ref="#PWR?"  Part="1"
-AR Path="/5BB6E330/5BB6E8F3" Ref="#PWR040"  Part="1"
-F 0 "#PWR040" H 4200 3800 50  0001 C CNN
+AR Path="/5BB6E330/5BB6E8F3" Ref="#PWR072"  Part="1"
+F 0 "#PWR072" H 4200 3800 50  0001 C CNN
 F 1 "+3.3V" H 4215 4123 50  0000 C CNN
 F 2 "" H 4200 3950 50  0001 C CNN
