File: pcb/SONAR-GPIO.sch (KiCad schematic (older format))
At the start: 57 parts, among them Q1 BSS138, Q10 BSS138, Q11 BSS138, Q12 BSS138, Q2 BSS138, Q3 BSS138, Q4 BSS138, Q5 BSS138, Q6 BSS138, Q7 BSS138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

Commit message: Connect some more wires
Parts:
- added S?: EG1218, digikey-footprints:Switch_Slide_11.6x4mm_EG1218, symbol dk_Slide-Switches:EG1218
Changed lines of the file:
@@
 Wire Wire Line
 	10700 1950 10700 3450
+$Comp
+L dk_Slide-Switches:EG1218 S?
+U 1 1 5BC0AE93
+P 1250 850
+F 0 "S?" H 1250 1129 50  0000 C CNN
+F 1 "EG1218" H 1250 1038 50  0000 C CNN
+F 2 "digikey-footprints:Switch_Slide_11.6x4mm_EG1218" H 1450 1050 50  0001 L CNN
+F 3 "http://spec_sheets.e-switch.com/specs/P040040.pdf" H 1450 1150 60  0001 L CNN
+F 4 "EG1903-ND" H 1450 1250 60  0001 L CNN "Digi-Key_PN"
+F 5 "EG1218" H 1450 1350 60  0001 L CNN "MPN"
+F 6 "Switches" H 1450 1450 60  0001 L CNN "Category"
+F 7 "Slide Switches" H 1450 1550 60  0001 L CNN "Family"
+F 8 "http://spec_sheets.e-switch.com/specs/P040040.pdf" H 1450 1650 60  0001 L CNN "DK_Datasheet_Link"
+F 9 "/product-detail/en/e-switch/EG1218/EG1903-ND/101726" H 1450 1750 60  0001 L CNN "DK_Detail_Page"
+F 10 "SWITCH SLIDE SPDT 200MA 30V" H 1450 1850 60  0001 L CNN "Description"
+F 11 "E-Switch" H 1450 1950 60  0001 L CNN "Manufacturer"
+F 12 "Active" H 1450 2050 60  0001 L CNN "Status"
+	1    1250 850
+	1    0    0    -1
+$EndComp
 $EndSCHEMATC

Commit message: Think it is somewhat finished
Parts:
- removed JP11, JP12, JP13, JP14, JP15, JP16, JP17, JP18, JP19, JP20, JP21, JP22, JP23, JP24, JP25, JP26, JP27, JP28: Jumper_NC_Dual, Connector_PinHeader_2.54mm:PinHeader_1x03_P2.54mm_Vertical, symbol Device:Jumper_NC_Dual
- removed Q3: BSS138, digikey-footprints:SOT-23-3, symbol Transistor_FET:BSS138
- removed R12, R13, R32, R33, R34, R35: 10k, Resistor_SMD:R_1206_3216Metric_Pad1.42x1.75mm_HandSolder, symbol Device:R
- removed S?: EG1218, digikey-footprints:Switch_Slide_11.6x4mm_EG1218, symbol dk_Slide-Switches:EG1218
- added Q2: BSS138, digikey-footprints:SOT-23-3, symbol Transistor_FET:BSS138
- added R10, R11, R14, R15, R16, R17: 10k, Resistor_SMD:R_1206_3216Metric_Pad1.42x1.75mm_HandSolder, symbol Device:R
- added SW10, SW11, SW3, SW4, SW5, SW6, SW7, SW8, SW9: SW_2xSPDT, localization-footprints:CAS-D20TB, symbol localization-symbols:SW_2xSPDT
- renumbered Q2 to Q3, R10 to R12, R11 to R13, R7 to R8, R6 to R9
Connections:
- net labels added: A1, A2, A3, A4, B1, B2, B3, B4, C1, C2, C3, C4
- net labels removed: AD1, AD2, AD3_RX, AD4_TX, BD1, BD2, BD3_RX, BD4_TX, C3_RX, CD1, CD2, CD4_TX
- wire segments 198 -> 153
