File: pcb/IMU.sch (KiCad schematic (older format))
At the start: 1 part, among them U3 IMU

Commit message: Finishe schematic, add netlist and start editing pcb design
Parts:
- U3: footprint (none) -> localization-footprints:IMU
Changed lines of the file:
@@
 F 0 "U3" V 6021 3622 50  0000 R CNN
 F 1 "IMU" V 5930 3622 50  0000 R CNN
-F 2 "" V 6150 3850 50  0001 C CNN
+F 2 "localization-footprints:IMU" V 6150 3850 50  0001 C CNN
 F 3 "" V 6150 3850 50  0001 C CNN
 	1    6000 3950

Commit message: Add IMU footprint
Parts:
- U3: footprint localization-footprints:IMU -> Adafruit BNO055:BNO055
Connections:
- net labels added: +3.3V
- net labels removed: VCC
Changed lines of the file:
@@
 $Descr A4 11693 8268
 encoding utf-8
-Sheet 8 10
+Sheet 7 10
 Title ""
 Date ""
@@
 F 0 "U3" V 6021 3622 50  0000 R CNN
 F 1 "IMU" V 5930 3622 50  0000 R CNN
-F 2 "localization-footprints:IMU" V 6150 3850 50  0001 C CNN
+F 2 "Adafruit BNO055:BNO055" V 6150 3850 50  0001 C CNN
 F 3 "" V 6150 3850 50  0001 C CNN
 	1    6000 3950
 	0    -1   -1   0
-$EndComp
-$Comp
-L power:VCC #PWR024
-U 1 1 5BB1BB96
-P 6250 3550
-F 0 "#PWR024" H 6250 3400 50  0001 C CNN
-F 1 "VCC" H 6267 3723 50  0000 C CNN
-F 2 "" H 6250 3550 50  0001 C CNN
-F 3 "" H 6250 3550 50  0001 C CNN
-	1    6250 3550
-	1    0    0    -1
 $EndComp
 $Comp
@@
 Wire Wire Line
 	6050 3550 6050 3650
-Wire Wire Line
-	6250 3550 6250 3650
 NoConn ~ 6150 3650
 NoConn ~ 6150 4300
@@
 NoConn ~ 5950 4300
 NoConn ~ 5850 4300
+$Comp
+L power:+3.3V #PWR0101
+U 1 1 5BAD3F69
+P 6250 3550
+F 0 "#PWR0101" H 6250 3400 50  0001 C CNN
+F 1 "+3.3V" H 6265 3723 50  0000 C CNN
+F 2 "" H 6250 3550 50  0001 C CNN
+F 3 "" H 6250 3550 50  0001 C CNN
+	1    6250 3550
+	1    0    0    -1
+$EndComp
+Wire Wire Line
+	6250 3650 6250 3550
 $EndSCHEMATC

Commit message: Add level shifters and jumpers and new gpio
Parts:
- added R8: 2.2k, Resistor_SMD:R_1206_3216Metric_Pad1.42x1.75mm_HandSolder, symbol Device:R
- added R9: 4.7k, Resistor_SMD:R_1206_3216Metric_Pad1.42x1.75mm_HandSolder, symbol Device:R
Connections:
- net labels added: INT
- wire segments 5 -> 10
- no-connect marks 5 -> 4
Changed lines of the file:
@@
 L localization-symbols:IMU U?
 U 1 1 5BB1BB38
-P 6000 3950
+P 6050 3900
 AR Path="/5BB1BB38" Ref="U?"  Part="1"
 AR Path="/5BB1BAF2/5BB1BB38" Ref="U3"  Part="1"
-F 0 "U3" V 6021 3622 50  0000 R CNN
-F 1 "IMU" V 5930 3622 50  0000 R CNN
-F 2 "Adafruit BNO055:BNO055" V 6150 3850 50  0001 C CNN
-F 3 "" V 6150 3850 50  0001 C CNN
-	1    6000 3950
-	0    -1   -1   0
+F 0 "U3" V 6071 3572 50  0000 R CNN
+F 1 "IMU" V 5980 3572 50  0000 R CNN
+F 2 "Adafruit BNO055:BNO055" V 6200 3800 50  0001 C CNN
+F 3 "" V 6200 3800 50  0001 C CNN
+	1    6050 3900
+	-1   0    0    1
 $EndComp
 $Comp
 L power:GND #PWR023
 U 1 1 5BB1BBFA
-P 6050 3550
-F 0 "#PWR023" H 6050 3300 50  0001 C CNN
-F 1 "GND" H 6055 3377 50  0000 C CNN
-F 2 "" H 6050 3550 50  0001 C CNN
-F 3 "" H 6050 3550 50  0001 C CNN
-	1    6050 3550
-	-1   0    0    1
+P 5650 3850
+F 0 "#PWR023" H 5650 3600 50  0001 C CNN
+F 1 "GND" H 5655 3677 50  0000 C CNN
+F 2 "" H 5650 3850 50  0001 C CNN
+F 3 "" H 5650 3850 50  0001 C CNN
+	1    5650 3850
+	0    1    1    0
 $EndComp
-Text HLabel 5750 3550 1    50   Input ~ 0
+Text HLabel 5650 4150 0    50   Input ~ 0
 RST
-Text HLabel 5850 3550 1    50   Input ~ 0
+Text HLabel 4750 4050 0    50   Input ~ 0
 SCL
-Text HLabel 5950 3550 1    50   Input ~ 0
+Text HLabel 4750 3950 0    50   Input ~ 0
 SDA
 Wire Wire Line
-	5750 3550 5750 3650
+	5650 4150 5750 4150
 Wire Wire Line
-	5850 3550 5850 3650
-Wire Wire Line
-	5950 3550 5950 3650
-Wire Wire Line
-	6050 3550 6050 3650
-NoConn ~ 6150 3650
-NoConn ~ 6150 4300
-NoConn ~ 6050 4300
-NoConn ~ 5950 4300
-NoConn ~ 5850 4300
+	5650 3850 5750 3850
+NoConn ~ 5750 3750
+NoConn ~ 6400 3750
+NoConn ~ 6400 3850
+NoConn ~ 6400 4050
 $Comp
 L power:+3.3V #PWR0101
 U 1 1 5BAD3F69
-P 6250 3550
-F 0 "#PWR0101" H 6250 3400 50  0001 C CNN
-F 1 "+3.3V" H 6265 3723 50  0000 C CNN
-F 2 "" H 6250 3550 50  0001 C CNN
-F 3 "" H 6250 3550 50  0001 C CNN
-	1    6250 3550
+P 5650 3650
+F 0 "#PWR0101" H 5650 3500 50  0001 C CNN
+F 1 "+3.3V" H 5665 3823 50  0000 C CNN
+F 2 "" H 5650 3650 50  0001 C CNN
+F 3 "" H 5650 3650 50  0001 C CNN
+	1    5650 3650
+	0    -1   -1   0
+$EndComp
+Wire Wire Line
+	5750 3650 5650 3650
+Text HLabel 6500 3950 2    50   Input ~ 0
+INT
+Wire Wire Line
+	6400 3950 6500 3950
+$Comp
+L Device:R R9
+U 1 1 5BB87CE6
+P 5150 3700
+F 0 "R9" H 5220 3746 50  0000 L CNN
+F 1 "4.7k" H 5220 3655 50  0000 L CNN
+F 2 "Resistor_SMD:R_1206_3216Metric_Pad1.42x1.75mm_HandSolder" V 5080 3700 50  0001 C CNN
+F 3 "~" H 5150 3700 50  0001 C CNN
+	1    5150 3700
+	1    0    0    -1
+$EndComp
+$Comp
+L Device:R R8
+U 1 1 5BB87D2C
+P 4850 3700
+F 0 "R8" H 4920 3746 50  0000 L CNN
+F 1 "2.2k" H 4920 3655 50  0000 L CNN
+F 2 "Resistor_SMD:R_1206_3216Metric_Pad1.42x1.75mm_HandSolder" V 4780 3700 50  0001 C CNN
+F 3 "~" H 4850 3700 50  0001 C CNN
+	1    4850 3700
 	1    0    0    -1
 $EndComp
 Wire Wire Line
-	6250 3650 6250 3550
+	4750 3950 4850 3950
+Wire Wire Line
+	4750 4050 5150 4050
+Wire Wire Line
+	4850 3850 4850 3950
+Connection ~ 4850 3950
+Wire Wire Line
+	4850 3950 5750 3950
+Wire Wire Line
+	5150 3850 5150 4050
+Connection ~ 5150 4050
+Wire Wire Line
+	5150 4050 5750 4050
+$Comp
+L DMPro17-rescue:+3.3V #PWR0103
+U 1 1 5BB87FE9
+P 4850 3550
+F 0 "#PWR0103" H 4850 3400 50  0001 C CNN
+F 1 "+3.3V" H 4865 3723 50  0000 C CNN
+F 2 "" H 4850 3550 50  0001 C CNN
+F 3 "" H 4850 3550 50  0001 C CNN
+	1    4850 3550
+	1    0    0    -1
+$EndComp
+$Comp
+L DMPro17-rescue:+3.3V #PWR0104
+U 1 1 5BB88125
+P 5150 3550
+F 0 "#PWR0104" H 5150 3400 50  0001 C CNN
+F 1 "+3.3V" H 5165 3723 50  0000 C CNN
+F 2 "" H 5150 3550 50  0001 C CNN
+F 3 "" H 5150 3550 50  0001 C CNN
+	1    5150 3550
+	1    0    0    -1
+$EndComp
 $EndSCHEMATC

Commit message: Think it is somewhat finished
Parts:
- renumbered R8 to R6, R9 to R7
Changed lines of the file:
@@
 $EndComp
 $Comp
-L power:GND #PWR023
+L power:GND #PWR024
 U 1 1 5BB1BBFA
 P 5650 3850
-F 0 "#PWR023" H 5650 3600 50  0001 C CNN
+F 0 "#PWR024" H 5650 3600 50  0001 C CNN
 F 1 "GND" H 5655 3677 50  0000 C CNN
 F 2 "" H 5650 3850 50  0001 C CNN
@@
 NoConn ~ 6400 4050
 $Comp
-L power:+3.3V #PWR0101
+L power:+3.3V #PWR023
 U 1 1 5BAD3F69
 P 5650 3650
-F 0 "#PWR0101" H 5650 3500 50  0001 C CNN
+F 0 "#PWR023" H 5650 3500 50  0001 C CNN
 F 1 "+3.3V" H 5665 3823 50  0000 C CNN
 F 2 "" H 5650 3650 50  0001 C CNN
@@
 	6400 3950 6500 3950
 $Comp
-L Device:R R9
+L Device:R R7
 U 1 1 5BB87CE6
 P 5150 3700
-F 0 "R9" H 5220 3746 50  0000 L CNN
+F 0 "R7" H 5220 3746 50  0000 L CNN
 F 1 "4.7k" H 5220 3655 50  0000 L CNN
 F 2 "Resistor_SMD:R_1206_3216Metric_Pad1.42x1.75mm_HandSolder" V 5080 3700 50  0001 C CNN
@@
 $EndComp
 $Comp
-L Device:R R8
+L Device:R R6
 U 1 1 5BB87D2C
 P 4850 3700
-F 0 "R8" H 4920 3746 50  0000 L CNN
+F 0 "R6" H 4920 3746 50  0000 L CNN
 F 1 "2.2k" H 4920 3655 50  0000 L CNN
 F 2 "Resistor_SMD:R_1206_3216Metric_Pad1.42x1.75mm_HandSolder" V 4780 3700 50  0001 C CNN
@@
 	5150 4050 5750 4050
 $Comp
-L DMPro17-rescue:+3.3V #PWR0103
+L DMPro17-rescue:+3.3V #PWR021
 U 1 1 5BB87FE9
 P 4850 3550
-F 0 "#PWR0103" H 4850 3400 50  0001 C CNN
+F 0 "#PWR021" H 4850 3400 50  0001 C CNN
 F 1 "+3.3V" H 4865 3723 50  0000 C CNN
 F 2 "" H 4850 3550 50  0001 C CNN
@@
 $EndComp
 $Comp
-L DMPro17-rescue:+3.3V #PWR0104
+L DMPro17-rescue:+3.3V #PWR022
 U 1 1 5BB88125
 P 5150 3550
-F 0 "#PWR0104" H 5150 3400 50  0001 C CNN
+F 0 "#PWR022" H 5150 3400 50  0001 C CNN
 F 1 "+3.3V" H 5165 3723 50  0000 C CNN
 F 2 "" H 5150 3550 50  0001 C CNN

Commit message: Fix pin silk and size of IMU
Parts:
- U3: footprint Adafruit BNO055:BNO055 -> Adafruit-BNO055-Breakout-PCB-master:BNO055
Changed lines of the file:
@@
 F 0 "U3" V 6071 3572 50  0000 R CNN
 F 1 "IMU" V 5980 3572 50  0000 R CNN
-F 2 "Adafruit BNO055:BNO055" V 6200 3800 50  0001 C CNN
+F 2 "Adafruit-BNO055-Breakout-PCB-master:BNO055" V 6200 3800 50  0001 C CNN
 F 3 "" V 6200 3800 50  0001 C CNN
 	1    6050 3900
